Commit message: Inital Fake YOLO, have bounding boxes being generated with debug image for SG, and dice
Added distortion coefficents correctly to leviathan gazebo cameras
Moved start gate model top to be at origin
Added pose sensors to start gate and dice 5

File: cusub_sim/Description/leviathan_description/urdf/snippets.xacro (robot description, xacro)
@@ -33,5 +33,4 @@
       <camera name="rgb_camera">
         <horizontal_fov>1.0397</horizontal_fov>
-        <vertical_fov>0.6443</vertical_fov>
         <image>
           <width>752</width>
@@ -43,4 +42,12 @@
           <far>300</far>
         </clip>
+        <distortion>
+          <k1>-0.360085</k1>
+          <k2>0.115116</k2>
+          <k3>0.0</k3>
+          <p1>0.007768</p1>
+          <p2>0.004616</p2>
+          <center>0.5 0.5</center>
+        </distortion>
       </camera>
       <plugin name="camera_controller" filename="libgazebo_ros_camera.so">
@@ -51,10 +58,9 @@
         <cameraInfoTopicName>camera_info</cameraInfoTopicName>
         <frameName>${frame}</frameName>
-        <hackBaseline>0.0</hackBaseline>
         <distortionK1>-0.360085</distortionK1>
         <distortionK2>0.115116</distortionK2>
-        <distortionK3>0.007768</distortionK3>
-        <distortionT1>0.004616</distortionT1>
-        <distortionT2>0.000000</distortionT2>
+        <distortionK3>0.000000</distortionK3>
+        <distortionT1>0.007768</distortionT1>
+        <distortionT2>0.004616</distortionT2>
       </plugin>
     </sensor>

File: cusub_sim/Gazebo_Sim/robosub_descriptions/urdf/Dice5.xacro (robot description, xacro)
@@ -1,5 +1,9 @@
-<robot
+<?xml version="1.0"?>
+<robot xmlns:xacro="http://www.ros.org/wiki/xacro"
   name="Dice5_robot">
-  <link name="Dice5/base_link">
+<!-- Loading file with sensor macros -->
+<xacro:include filename="$(find uuv_sensor_ros_plugins)/urdf/sensor_snippets.xacro"/>
+<xacro:macro name="dice5_base" params="namespace">
+  <link name="${namespace}/base_link">
     <inertial>
       <origin
@@ -35,4 +39,5 @@
     </collision>
   </link>
+  <xacro:default_pose_3d namespace="${namespace}" parent_link="${namespace}/base_link" />
   <link name = "Dice5/string_link">
   <inertial>
@@ -87,5 +92,5 @@
       xyz="0.1143 -0.1143 -0.2286"
       rpy="0 0 0" />
-    <parent link="Dice5/base_link"/>
+    <parent link="${namespace}/base_link"/>
     <child link="Dice5/string_link"/>
   </joint>
@@ -102,5 +107,5 @@
     <flow_velocity_topic>hydrodynamics/current_velocity</flow_velocity_topic>
     <debug>0</debug>
-    <link name="Dice5/base_link">
+    <link name="${namespace}/base_link">
         <fluid_density>1028</fluid_density>
         <flow_velocity_topic>hydrodynamics/current_velocity</flow_velocity_topic>
@@ -121,3 +126,5 @@
     </plugin>
   </gazebo>
+</xacro:macro>
+<xacro:dice5_base namespace="$(arg namespace)"/>
 </robot>

File: cusub_sim/Gazebo_Sim/robosub_descriptions/urdf/StartGate.xacro (robot description, xacro)
@@ -1,6 +1,10 @@
-<robot
+<?xml version="1.0"?>
+<robot xmlns:xacro="http://www.ros.org/wiki/xacro"
   name="StartGate_robot">
+<!-- Loading file with sensor macros -->
+<xacro:include filename="$(find uuv_sensor_ros_plugins)/urdf/sensor_snippets.xacro"/>
+<xacro:macro name="startgate_base" params="namespace">
   <link
-    name="StartGate_link">
+    name="${namespace}/base_link">
     <inertial>
       <origin
@@ -34,6 +38,12 @@
     </collision>
   </link>
-  <gazebo reference="StartGate_link">
+  <xacro:default_pose_3d namespace="${namespace}" parent_link="${namespace}/base_link" />
+  <gazebo reference="${namespace}/base_link">
       <turnGravityOff>true</turnGravityOff>
   </gazebo>
+  <gazebo>
+      <static>true</static>
+  </gazebo>
+</xacro:macro>
+<xacro:startgate_base namespace="$(arg namespace)"/>
 </robot>

Commit message: Changed levithan camera macros so we seperate the downcam Inflated occam FoV to compensate for gazebo crop Added publishing of darknet detections to FakeYOLO

File: cusub_sim/Description/leviathan_description/urdf/snippets.xacro (robot description, xacro)
@@ -1,5 +1,5 @@
 <?xml version="1.0"?>
 <robot xmlns:xacro="http://www.ros.org/wiki/xacro">
-  <xacro:macro name="camera_macro" params="robot_namespace camera_id frame *axis *origin">
+  <xacro:macro name="occam_camera_macro" params="robot_namespace camera_id frame *axis *origin">
   <!--camera_link-->
   <link name="${robot_namespace}/camera_${camera_id}">
@@ -32,5 +32,12 @@
       <update_rate>30.0</update_rate>
       <camera name="rgb_camera">
-        <horizontal_fov>1.0397</horizontal_fov>
+        <!--
+          The correct FOV is 1.0397, but because of gazebo distortion crop we
+           need to inflate it by 20% so it ends up the correct size
+          This will unfortunatly make it report a faulty camera matrix
+          TODO see if camera intrinsics propertys are working maybe we
+           can override
+        -->
+        <horizontal_fov>1.24764</horizontal_fov>
         <image>
           <width>752</width>
@@ -63,4 +70,70 @@
         <distortionT1>0.007768</distortionT1>
         <distortionT2>0.004616</distortionT2>
+      </plugin>
+    </sensor>
+  </gazebo>
+  </xacro:macro>
+  <xacro:macro name="downcam_camera_macro" params="robot_namespace camera_id frame *axis *origin">
+  <!--camera_link-->
+  <link name="${robot_namespace}/camera_${camera_id}">
+    <collision>
+      <origin xyz="0 0 0" rpy="0 0 0"/>
+      <geometry>
+        <!--mesh filename="package://simple_arm/meshes/camera.dae"/-->
+        <sphere radius="0.01"/>
+      </geometry>
+    </collision>
+    <visual>
+      <origin xyz="0 0 0" rpy="0 0 0"/>
+      <geometry>
+        <!--mesh filename="package://simple_arm/meshes/camera.dae"/-->
+        <sphere radius="0.01"/>
+      </geometry>
+      <material name="red">
+        <color rgba="1.0 0 0 1.0"/>
+      </material>
+    </visual>
+  </link>
+  <joint name="${robot_namespace}/camera_${camera_id}_joint" type="fixed">
+    <xacro:insert_block name="axis" />
+    <xacro:insert_block name="origin" />
+    <parent link="${namespace}/base_link"/>
+    <child link="${robot_namespace}/camera_${camera_id}"/>
+  </joint>
+  <gazebo reference="${robot_namespace}/camera_${camera_id}">
+    <sensor type="camera" name="rgb_camera">
+      <update_rate>30.0</update_rate>
+      <camera name="rgb_camera">
+        <horizontal_fov>2.18166</horizontal_fov>
+        <image>
+          <width>752</width>
+          <height>480</height>
+          <format>R8G8B8</format>
+        </image>
+        <clip>
+          <near>0.02</near>
+          <far>300</far>
+        </clip>
+        <distortion>
+          <k1>0</k1>
+          <k2>0</k2>
+          <k3>0</k3>
+          <p1>0</p1>
+          <p2>0</p2>
+          <center>0.5 0.5</center>
+        </distortion>
+      </camera>
+      <plugin name="camera_controller" filename="libgazebo_ros_camera.so">
+        <alwaysOn>true</alwaysOn>
+        <updateRate>0.0</updateRate>
+        <cameraName>camera_${camera_id}</cameraName>
+        <imageTopicName>image_raw</imageTopicName>
+        <cameraInfoTopicName>camera_info</cameraInfoTopicName>
+        <frameName>${frame}</frameName>
+        <distortionK1>0</distortionK1>
+        <distortionK2>0</distortionK2>
+        <distortionK3>0</distortionK3>
+        <distortionT1>0</distortionT1>
+        <distortionT2>0</distortionT2>
       </plugin>
     </sensor>
