Commit message: Added dice 1 and 2 to divewell simulation

File: cusub_sim/robosub_descriptions/urdf/Dice1.xacro (robot description, xacro)
@@ -1,8 +1,8 @@
 <?xml version="1.0"?>
 <robot xmlns:xacro="http://www.ros.org/wiki/xacro"
-  name="Dice6_robot">
+  name="dice1_robot">
 <!-- Loading file with sensor macros -->
 <xacro:include filename="$(find uuv_sensor_ros_plugins)/urdf/sensor_snippets.xacro"/>
-<xacro:macro name="dice6_base" params="namespace">
+<xacro:macro name="dice1_base" params="namespace">
   <link name="${namespace}/base_link">
     <inertial>
@@ -26,5 +26,5 @@
       <geometry>
         <mesh
-          filename="package://robosub_descriptions/meshes/Dice6.dae" />
+          filename="package://robosub_descriptions/meshes/Dice1.dae" />
       </geometry>
     </visual>
@@ -40,5 +40,5 @@
   </link>
   <xacro:default_pose_3d namespace="${namespace}" parent_link="${namespace}/base_link" />
-  <link name = "Dice6/string_link">
+  <link name = "dice1/string_link">
   <inertial>
     <origin
@@ -56,5 +56,5 @@
   </inertial>
   </link>
-  <link name = "Dice6/anchor_link">
+  <link name = "dice1/anchor_link">
     <inertial>
       <origin
@@ -88,17 +88,17 @@
     </collision>
   </link>
-  <joint name="Dice6/base_joint" type="continuous">
+  <joint name="dice1/base_joint" type="continuous">
     <origin
       xyz="0.1143 -0.1143 -0.2286"
       rpy="0 0 0" />
     <parent link="${namespace}/base_link"/>
-    <child link="Dice6/string_link"/>
+    <child link="dice1/string_link"/>
   </joint>
-  <joint name="Dice6/anchor_joint" type="continuous">
+  <joint name="dice1/anchor_joint" type="continuous">
     <origin
-      xyz="0 0 -2.2"
+      xyz="0 0 -2.3"
       rpy="0 0 0" />
-    <parent link="Dice6/string_link"/>
-    <child link="Dice6/anchor_link"/>
+    <parent link="dice1/string_link"/>
+    <child link="dice1/anchor_link"/>
   </joint>
   <gazebo>
@@ -127,4 +127,4 @@
   </gazebo>
 </xacro:macro>
-<xacro:dice6_base namespace="$(arg namespace)"/>
+<xacro:dice1_base namespace="$(arg namespace)"/>
 </robot>

File: cusub_sim/robosub_descriptions/urdf/Dice2.xacro (robot description, xacro)
@@ -1,8 +1,8 @@
 <?xml version="1.0"?>
 <robot xmlns:xacro="http://www.ros.org/wiki/xacro"
-  name="Dice6_robot">
+  name="dice2_robot">
 <!-- Loading file with sensor macros -->
 <xacro:include filename="$(find uuv_sensor_ros_plugins)/urdf/sensor_snippets.xacro"/>
-<xacro:macro name="dice6_base" params="namespace">
+<xacro:macro name="dice2_base" params="namespace">
   <link name="${namespace}/base_link">
     <inertial>
@@ -26,5 +26,5 @@
       <geometry>
         <mesh
-          filename="package://robosub_descriptions/meshes/Dice6.dae" />
+          filename="package://robosub_descriptions/meshes/Dice2.dae" />
       </geometry>
     </visual>
@@ -40,5 +40,5 @@
   </link>
   <xacro:default_pose_3d namespace="${namespace}" parent_link="${namespace}/base_link" />
-  <link name = "Dice6/string_link">
+  <link name = "dice2/string_link">
   <inertial>
     <origin
@@ -56,5 +56,5 @@
   </inertial>
   </link>
-  <link name = "Dice6/anchor_link">
+  <link name = "dice2/anchor_link">
     <inertial>
       <origin
@@ -88,17 +88,17 @@
     </collision>
   </link>
-  <joint name="Dice6/base_joint" type="continuous">
+  <joint name="dice2/base_joint" type="continuous">
     <origin
       xyz="0.1143 -0.1143 -0.2286"
       rpy="0 0 0" />
     <parent link="${namespace}/base_link"/>
-    <child link="Dice6/string_link"/>
+    <child link="dice2/string_link"/>
   </joint>
-  <joint name="Dice6/anchor_joint" type="continuous">
+  <joint name="dice2/anchor_joint" type="continuous">
     <origin
-      xyz="0 0 -2.2"
+      xyz="0 0 -1.6"
       rpy="0 0 0" />
-    <parent link="Dice6/string_link"/>
-    <child link="Dice6/anchor_link"/>
+    <parent link="dice2/string_link"/>
+    <child link="dice2/anchor_link"/>
   </joint>
   <gazebo>
@@ -127,4 +127,4 @@
   </gazebo>
 </xacro:macro>
-<xacro:dice6_base namespace="$(arg namespace)"/>
+<xacro:dice2_base namespace="$(arg namespace)"/>
 </robot>

File: cusub_sim/robosub_descriptions/urdf/Dice5.xacro (robot description, xacro)
@@ -1,5 +1,9 @@
-<robot
+<?xml version="1.0"?>
+<robot xmlns:xacro="http://www.ros.org/wiki/xacro"
   name="Dice5_robot">
-  <link name="Dice5/base_link">
+<!-- Loading file with sensor macros -->
+<xacro:include filename="$(find uuv_sensor_ros_plugins)/urdf/sensor_snippets.xacro"/>
+<xacro:macro name="dice5_base" params="namespace">
+  <link name="${namespace}/base_link">
     <inertial>
       <origin
@@ -35,4 +39,5 @@
     </collision>
   </link>
+  <xacro:default_pose_3d namespace="${namespace}" parent_link="${namespace}/base_link" />
   <link name = "Dice5/string_link">
   <inertial>
@@ -87,10 +92,10 @@
       xyz="0.1143 -0.1143 -0.2286"
       rpy="0 0 0" />
-    <parent link="Dice5/base_link"/>
+    <parent link="${namespace}/base_link"/>
     <child link="Dice5/string_link"/>
   </joint>
   <joint name="Dice5/anchor_joint" type="continuous">
     <origin
-      xyz="0 0 -2"
+      xyz="0 0 -1.8"
       rpy="0 0 0" />
     <parent link="Dice5/string_link"/>
@@ -102,5 +107,5 @@
     <flow_velocity_topic>hydrodynamics/current_velocity</flow_velocity_topic>
     <debug>0</debug>
-    <link name="Dice5/base_link">
+    <link name="${namespace}/base_link">
         <fluid_density>1028</fluid_density>
         <flow_velocity_topic>hydrodynamics/current_velocity</flow_velocity_topic>
@@ -121,3 +126,5 @@
     </plugin>
   </gazebo>
+</xacro:macro>
+<xacro:dice5_base namespace="$(arg namespace)"/>
 </robot>
