Commit message: Restructured robosub descriptions closes #14

File: cusub_sim/robosub_descriptions/models/Dice1/Dice1.xacro (robot description, xacro)
@@ -1,8 +1,8 @@
 <?xml version="1.0"?>
 <robot xmlns:xacro="http://www.ros.org/wiki/xacro"
-  name="Dice5_robot">
+  name="dice1_robot">
 <!-- Loading file with sensor macros -->
 <xacro:include filename="$(find uuv_sensor_ros_plugins)/urdf/sensor_snippets.xacro"/>
-<xacro:macro name="dice5_base" params="namespace">
+<xacro:macro name="dice1_base" params="namespace">
   <link name="${namespace}/base_link">
     <inertial>
@@ -26,5 +26,5 @@
       <geometry>
         <mesh
-          filename="package://robosub_descriptions/meshes/Dice5.dae" />
+          filename="package://robosub_descriptions/models/Dice1/Dice1.dae" />
       </geometry>
     </visual>
@@ -35,10 +35,10 @@
       <geometry>
         <mesh
-          filename="package://robosub_descriptions/meshes/Dice.stl" />
+          filename="package://robosub_descriptions/models/shared/Dice.stl" />
       </geometry>
     </collision>
   </link>
   <xacro:default_pose_3d namespace="${namespace}" parent_link="${namespace}/base_link" />
-  <link name = "Dice5/string_link">
+  <link name = "dice1/string_link">
   <inertial>
     <origin
@@ -56,5 +56,5 @@
   </inertial>
   </link>
-  <link name = "Dice5/anchor_link">
+  <link name = "dice1/anchor_link">
     <inertial>
       <origin
@@ -88,17 +88,17 @@
     </collision>
   </link>
-  <joint name="Dice5/base_joint" type="continuous">
+  <joint name="dice1/base_joint" type="continuous">
     <origin
       xyz="0.1143 -0.1143 -0.2286"
       rpy="0 0 0" />
     <parent link="${namespace}/base_link"/>
-    <child link="Dice5/string_link"/>
+    <child link="dice1/string_link"/>
   </joint>
-  <joint name="Dice5/anchor_joint" type="continuous">
+  <joint name="dice1/anchor_joint" type="continuous">
     <origin
-      xyz="0 0 -1.8"
+      xyz="0 0 -2.3"
       rpy="0 0 0" />
-    <parent link="Dice5/string_link"/>
-    <child link="Dice5/anchor_link"/>
+    <parent link="dice1/string_link"/>
+    <child link="dice1/anchor_link"/>
   </joint>
   <gazebo>
@@ -127,4 +127,4 @@
   </gazebo>
 </xacro:macro>
-<xacro:dice5_base namespace="$(arg namespace)"/>
+<xacro:dice1_base namespace="$(arg namespace)"/>
 </robot>

File: cusub_sim/robosub_descriptions/models/Dice2/Dice2.xacro (robot description, xacro)
@@ -26,5 +26,5 @@
       <geometry>
         <mesh
-          filename="package://robosub_descriptions/meshes/Dice2.dae" />
+          filename="package://robosub_descriptions/models/Dice2/Dice2.dae" />
       </geometry>
     </visual>
@@ -35,5 +35,5 @@
       <geometry>
         <mesh
-          filename="package://robosub_descriptions/meshes/Dice.stl" />
+          filename="package://robosub_descriptions/models/shared/Dice.stl" />
       </geometry>
     </collision>

File: cusub_sim/robosub_descriptions/models/Dice5/Dice5.xacro (robot description, xacro)
@@ -1,8 +1,8 @@
 <?xml version="1.0"?>
 <robot xmlns:xacro="http://www.ros.org/wiki/xacro"
-  name="dice1_robot">
+  name="Dice5_robot">
 <!-- Loading file with sensor macros -->
 <xacro:include filename="$(find uuv_sensor_ros_plugins)/urdf/sensor_snippets.xacro"/>
-<xacro:macro name="dice1_base" params="namespace">
+<xacro:macro name="dice5_base" params="namespace">
   <link name="${namespace}/base_link">
     <inertial>
@@ -26,5 +26,5 @@
       <geometry>
         <mesh
-          filename="package://robosub_descriptions/meshes/Dice1.dae" />
+          filename="package://robosub_descriptions/models/Dice5/Dice5.dae" />
       </geometry>
     </visual>
@@ -35,10 +35,10 @@
       <geometry>
         <mesh
-          filename="package://robosub_descriptions/meshes/Dice.stl" />
+          filename="package://robosub_descriptions/models/shared/Dice.stl" />
       </geometry>
     </collision>
   </link>
   <xacro:default_pose_3d namespace="${namespace}" parent_link="${namespace}/base_link" />
-  <link name = "dice1/string_link">
+  <link name = "Dice5/string_link">
   <inertial>
     <origin
@@ -56,5 +56,5 @@
   </inertial>
   </link>
-  <link name = "dice1/anchor_link">
+  <link name = "Dice5/anchor_link">
     <inertial>
       <origin
@@ -88,17 +88,17 @@
     </collision>
   </link>
-  <joint name="dice1/base_joint" type="continuous">
+  <joint name="Dice5/base_joint" type="continuous">
     <origin
       xyz="0.1143 -0.1143 -0.2286"
       rpy="0 0 0" />
     <parent link="${namespace}/base_link"/>
-    <child link="dice1/string_link"/>
+    <child link="Dice5/string_link"/>
   </joint>
-  <joint name="dice1/anchor_joint" type="continuous">
+  <joint name="Dice5/anchor_joint" type="continuous">
     <origin
-      xyz="0 0 -2.3"
+      xyz="0 0 -1.8"
       rpy="0 0 0" />
-    <parent link="dice1/string_link"/>
-    <child link="dice1/anchor_link"/>
+    <parent link="Dice5/string_link"/>
+    <child link="Dice5/anchor_link"/>
   </joint>
   <gazebo>
@@ -127,4 +127,4 @@
   </gazebo>
 </xacro:macro>
-<xacro:dice1_base namespace="$(arg namespace)"/>
+<xacro:dice5_base namespace="$(arg namespace)"/>
 </robot>

File: cusub_sim/robosub_descriptions/models/Dice6/Dice6.xacro (robot description, xacro)
@@ -26,5 +26,5 @@
       <geometry>
         <mesh
-          filename="package://robosub_descriptions/meshes/Dice6.dae" />
+          filename="package://robosub_descriptions/models/Dice6/Dice6.dae" />
       </geometry>
     </visual>
@@ -35,5 +35,5 @@
       <geometry>
         <mesh
-          filename="package://robosub_descriptions/meshes/Dice.stl" />
+          filename="package://robosub_descriptions/models/shared/Dice.stl" />
       </geometry>
     </collision>
