Commit message: Added dice 1 and 2 to divewell simulation (#63)
* Added dice 1 and 2 to divewell simulation

* Restructured robosub descriptions
closes #14

File: cusub_sim/robosub_descriptions/models/Dice2/Dice2.xacro (robot description, xacro)
@@ -1,5 +1,9 @@
-<robot
-  name="Dice5_robot">
-  <link name="Dice5/base_link">
+<?xml version="1.0"?>
+<robot xmlns:xacro="http://www.ros.org/wiki/xacro"
+  name="dice2_robot">
+<!-- Loading file with sensor macros -->
+<xacro:include filename="$(find uuv_sensor_ros_plugins)/urdf/sensor_snippets.xacro"/>
+<xacro:macro name="dice2_base" params="namespace">
+  <link name="${namespace}/base_link">
     <inertial>
       <origin
@@ -22,5 +26,5 @@
       <geometry>
         <mesh
-          filename="package://robosub_descriptions/meshes/Dice5.dae" />
+          filename="package://robosub_descriptions/models/Dice2/Dice2.dae" />
       </geometry>
     </visual>
@@ -31,9 +35,10 @@
       <geometry>
         <mesh
-          filename="package://robosub_descriptions/meshes/Dice.stl" />
+          filename="package://robosub_descriptions/models/shared/Dice.stl" />
       </geometry>
     </collision>
   </link>
-  <link name = "Dice5/string_link">
+  <xacro:default_pose_3d namespace="${namespace}" parent_link="${namespace}/base_link" />
+  <link name = "dice2/string_link">
   <inertial>
     <origin
@@ -51,5 +56,5 @@
   </inertial>
   </link>
-  <link name = "Dice5/anchor_link">
+  <link name = "dice2/anchor_link">
     <inertial>
       <origin
@@ -83,17 +88,17 @@
     </collision>
   </link>
-  <joint name="Dice5/base_joint" type="continuous">
+  <joint name="dice2/base_joint" type="continuous">
     <origin
       xyz="0.1143 -0.1143 -0.2286"
       rpy="0 0 0" />
-    <parent link="Dice5/base_link"/>
-    <child link="Dice5/string_link"/>
+    <parent link="${namespace}/base_link"/>
+    <child link="dice2/string_link"/>
   </joint>
-  <joint name="Dice5/anchor_joint" type="continuous">
+  <joint name="dice2/anchor_joint" type="continuous">
     <origin
-      xyz="0 0 -2"
+      xyz="0 0 -1.6"
       rpy="0 0 0" />
-    <parent link="Dice5/string_link"/>
-    <child link="Dice5/anchor_link"/>
+    <parent link="dice2/string_link"/>
+    <child link="dice2/anchor_link"/>
   </joint>
   <gazebo>
@@ -102,5 +107,5 @@
     <flow_velocity_topic>hydrodynamics/current_velocity</flow_velocity_topic>
     <debug>0</debug>
-    <link name="Dice5/base_link">
+    <link name="${namespace}/base_link">
         <fluid_density>1028</fluid_density>
         <flow_velocity_topic>hydrodynamics/current_velocity</flow_velocity_topic>
@@ -121,3 +126,5 @@
     </plugin>
   </gazebo>
+</xacro:macro>
+<xacro:dice2_base namespace="$(arg namespace)"/>
 </robot>

File: cusub_sim/robosub_descriptions/models/Dice6/Dice6.xacro (robot description, xacro)
@@ -26,5 +26,5 @@
       <geometry>
         <mesh
-          filename="package://robosub_descriptions/meshes/Dice6.dae" />
+          filename="package://robosub_descriptions/models/Dice6/Dice6.dae" />
       </geometry>
     </visual>
@@ -35,5 +35,5 @@
       <geometry>
         <mesh
-          filename="package://robosub_descriptions/meshes/Dice.stl" />
+          filename="package://robosub_descriptions/models/shared/Dice.stl" />
       </geometry>
     </collision>
@@ -97,5 +97,5 @@
   <joint name="Dice6/anchor_joint" type="continuous">
     <origin
-      xyz="0 0 -1.75"
+      xyz="0 0 -2.2"
       rpy="0 0 0" />
     <parent link="Dice6/string_link"/>

File: cusub_sim/robosub_descriptions/models/GoldChip/GoldChip.xacro (robot description, xacro)
@@ -22,5 +22,5 @@
       <geometry>
         <mesh
-          filename="package://robosub_descriptions/meshes/goldchip_base_link.stl" />
+          filename="package://robosub_descriptions/models/GoldChip/goldchip_base_link.stl" />
       </geometry>
       <material
@@ -36,5 +36,5 @@
       <geometry>
         <mesh
-          filename="package://robosub_descriptions/meshes/goldchip_base_link.stl" />
+          filename="package://robosub_descriptions/models/GoldChip/goldchip_base_link.stl" />
       </geometry>
     </collision>
@@ -62,5 +62,5 @@
       <geometry>
         <mesh
-          filename="package://robosub_descriptions/meshes/goldchip_button_holder_link.stl" />
+          filename="package://robosub_descriptions/models/GoldChip/goldchip_button_holder_link.stl" />
       </geometry>
       <material
@@ -111,5 +111,5 @@
       <geometry>
         <mesh
-          filename="package://robosub_descriptions/meshes/GoldChipButton.dae" />
+          filename="package://robosub_descriptions/models/GoldChip/GoldChipButton.dae" />
       </geometry>
       <material
@@ -125,5 +125,5 @@
       <geometry>
         <mesh
-          filename="package://robosub_descriptions/meshes/goldchip_button_link.stl" />
+          filename="package://robosub_descriptions/models/GoldChip/goldchip_button_link.stl" />
       </geometry>
     </collision>

File: cusub_sim/robosub_descriptions/models/PathMarker/PathMarker.xacro (robot description, xacro)
@@ -23,5 +23,5 @@
       <geometry>
         <mesh
-          filename="package://robosub_descriptions/meshes/PathMarker.dae" />
+          filename="package://robosub_descriptions/models/PathMarker/PathMarker.dae" />
       </geometry>
     </visual>
@@ -32,5 +32,5 @@
       <geometry>
         <mesh
-          filename="package://robosub_descriptions/meshes/PathMarker.stl" />
+          filename="package://robosub_descriptions/models/PathMarker/PathMarker.stl" />
       </geometry>
     </collision>

File: cusub_sim/robosub_descriptions/models/Roulette/Roulette.xacro (robot description, xacro)
@@ -23,5 +23,5 @@
       <geometry>
         <mesh
-          filename="package://robosub_descriptions/meshes/Roulette.dae" />
+          filename="package://robosub_descriptions/models/Roulette/Roulette.dae" />
       </geometry>
     </visual>
@@ -32,5 +32,5 @@
       <geometry>
         <mesh
-          filename="package://robosub_descriptions/meshes/Roulette.stl" />
+          filename="package://robosub_descriptions/models/Roulette/Roulette.stl" />
       </geometry>
     </collision>

File: cusub_sim/robosub_descriptions/models/Roulette_spin/Roulette_spin.xacro (robot description, xacro)
@@ -9,5 +9,5 @@
       <origin xyz="0 0 0" rpy="0 0 0" />
       <geometry>
-        <mesh filename="package://robosub_descriptions/meshes/Roulette_base.stl" />
+        <mesh filename="package://robosub_descriptions/models/Roulette_spin/Roulette_base.stl" />
       </geometry>
       <material
@@ -19,5 +19,5 @@
       <origin xyz="0 0 0" rpy="0 0 0" />
       <geometry>
-        <mesh filename="package://robosub_descriptions/meshes/Roulette_base.stl" />
+        <mesh filename="package://robosub_descriptions/models/Roulette_spin/Roulette_base.stl" />
       </geometry>
     </collision>
@@ -36,5 +36,5 @@
       <origin xyz="0 0 0" rpy="0 0 0" />
       <geometry>
-        <mesh filename="package://robosub_descriptions/meshes/Roulette_table.dae" />
+        <mesh filename="package://robosub_descriptions/models/Roulette_spin/Roulette_table.dae" />
       </geometry>
     </visual>
@@ -42,5 +42,5 @@
       <origin xyz="0 0 0" rpy="0 0 0" />
       <geometry>
-        <mesh filename="package://robosub_descriptions/meshes/Roulette_table.stl" />
+        <mesh filename="package://robosub_descriptions/models/Roulette_spin/Roulette_table.stl" />
       </geometry>
     </collision>

File: cusub_sim/robosub_descriptions/models/StartGate/StartGate.xacro (robot description, xacro)
@@ -22,5 +22,5 @@
         rpy="0 0 0" />
       <geometry>
-        <mesh filename="package://robosub_descriptions/meshes/StartGate.dae" />
+        <mesh filename="package://robosub_descriptions/models/StartGate/StartGate.dae" />
       </geometry>
     </visual>
@@ -30,5 +30,5 @@
         rpy="0 0 0" />
       <geometry>
-        <mesh filename="package://robosub_descriptions/meshes/StartGate.dae" />
+        <mesh filename="package://robosub_descriptions/models/StartGate/StartGate.dae" />
       </geometry>
     </collision>
