Commit message: Completed physical model

File: cusub_sim/triton_description/urdf/actuators.xacro (robot description, xacro)
@@ -11,5 +11,5 @@
     <xacro:thruster_macro robot_namespace="${namespace}" thruster_id="0">
         <axis xyz="1 0 0"/>
-        <origin xyz="0.073152 -0.281686 0.032258" rpy="0 0 0" />
+        <origin xyz="0 -0.281686 0" rpy="0 0 0" />
     </xacro:thruster_macro>
     <!-- Left Motor -->
@@ -17,35 +17,35 @@
         <axis xyz="1 0 0"/>
         <!-- zxy -->
-        <origin xyz="0.073152 0.281686 0.032258" rpy="0 0 0" />
+        <origin xyz="0 0.281686 0" rpy="0 0 0" />
     </xacro:thruster_macro>
     <!-- Front Left Motor -->
     <xacro:thruster_macro robot_namespace="${namespace}" thruster_id="2">
         <axis xyz="1 0 0"/>
-    <origin xyz="0.37084 0.163068 -0.078486 " rpy="0 -1.5707963 0" />
+    <origin xyz="0.20284 0.199 0" rpy="0 -1.5707963 0" />
     </xacro:thruster_macro>
     <!-- Front Right Motor -->
     <xacro:thruster_macro robot_namespace="${namespace}" thruster_id="3">
         <axis xyz="1 0 0"/>
-    <origin xyz="0.37084 -0.163068 -0.078486" rpy="0 -1.5707963 0" />
+    <origin xyz="0.20284 -0.199 0" rpy="0 -1.5707963 0" />
     </xacro:thruster_macro>
     <!-- Back Left Motor -->
     <xacro:thruster_macro robot_namespace="${namespace}" thruster_id="4">
         <axis xyz="1 0 0"/>
-    <origin xyz="-0.38481 0.163068 -0.078486" rpy="0 -1.5707963 0" />
+    <origin xyz="-0.20481 0.199 0" rpy="0 -1.5707963 0" />
     </xacro:thruster_macro>
     <!-- Back Right Motor -->
     <xacro:thruster_macro robot_namespace="${namespace}" thruster_id="5">
         <axis xyz="1 0 0"/>
-    <origin xyz="-0.38481 -0.163068  -0.078486" rpy="0 -1.5707963 0" />
+    <origin xyz="-0.20481 -0.199 0" rpy="0 -1.5707963 0" />
     </xacro:thruster_macro>
     <!-- Front Motor -->
     <xacro:thruster_macro robot_namespace="${namespace}" thruster_id="6">
         <axis xyz="1 0 0"/>
-    <origin xyz="0.439166 -0.007874 -0.060706" rpy="0 0 -1.5707963" />
+    <origin xyz="0.289166 0 -0.010706" rpy="0 0 -1.5707963" />
     </xacro:thruster_macro>
     <!-- Back Motor -->
     <xacro:thruster_macro robot_namespace="${namespace}" thruster_id="7">
         <axis xyz="1 0 0"/>
-    <origin xyz="-0.453136 -0.007874 -0.060706" rpy="0 0 -1.5707963" />
+    <origin xyz="-0.289166 0 -0.010706" rpy="0 0 -1.5707963" />
     </xacro:thruster_macro>
 </robot>

File: cusub_sim/triton_description/urdf/base.xacro (robot description, xacro)
@@ -26,9 +26,9 @@
     Open the meshes for the RexROV vehicle in Blender to see an example on the mesh placement.
   -->
-  <xacro:property name="visual_mesh_file" value="file://$(find triton_description)/meshes/TritonMesh.stl"/>
+  <xacro:property name="visual_mesh_file" value="file://$(find triton_description)/meshes/TritonMesh.STL"/>
   <!-- Collision geometry mesh, usually in STL format (it is recommended to keep
   this geometry as simple as possible to improve the performance the physics engine
   regarding the computation of collision forces) -->
-  <xacro:property name="collision_mesh_file" value="file://$(find triton_description)/meshes/TritonMesh.stl"/>
+  <xacro:property name="collision_mesh_file" value="file://$(find triton_description)/meshes/TritonMesh.STL"/>
   <!-- Vehicle macro -->
   <xacro:macro name="triton_base" params="namespace *gazebo">

File: cusub_sim/triton_description/urdf/sensors.xacro (robot description, xacro)
@@ -20,5 +20,5 @@
   <xacro:ocam_camera_macro robot_namespace="${namespace}" camera_id="0" frame="ocam0_frame">
     <axis xyz="0 0 0" />
-    <origin xyz="0.055 0 0.22" rpy="0 -0.785398 0"/>
-  </xacro:occam_camera_macro>
+    <origin xyz="0.06 0 -0.05" rpy="0 -0.785398 0"/>
+  </xacro:ocam_camera_macro>
 </robot>
