Commit message: Tweaked Triton parameters for reasonable simulation

File: cusub_sim/triton_description/urdf/base.xacro (robot description, xacro)
@@ -12,8 +12,8 @@
     Vehicle's parameters (remember to enter the model parameters below)
   -->
-  <xacro:property name="x_size" value="0.5"/>
-  <xacro:property name="y_size"  value="0.5"/>
-  <xacro:property name="z_size" value="0.5"/>
-  <xacro:property name="mass" value="10"/>
+  <xacro:property name="x_size" value="0.25"/>
+  <xacro:property name="y_size"  value="0.25"/>
+  <xacro:property name="z_size" value="0.25"/>
+  <xacro:property name="mass" value="3"/>
   <!-- Center of gravity -->
   <xacro:property name="cog" value="0 0 0"/>

File: cusub_sim/triton_description/urdf/gazebo.xacro (robot description, xacro)
@@ -2,11 +2,11 @@
 <robot xmlns:xacro="http://www.ros.org/wiki/xacro">
     <!-- Center of buoyancy -->
-    <xacro:property name="triton_cob" value="0 0 0"/>
+    <xacro:property name="triton_cob" value="0 0 0.2"/>
     <!-- Vehicle's actual volume (Gazebo cannot compute the volume out of the mesh) -->
-    <xacro:property name="triton_volume" value="0"/>
+    <xacro:property name="triton_volume" value="0.00439"/>
     <!-- Describing the dimensions of the vehicle's bounding box -->
-    <xacro:property name="triton_length" value="0.5"/>
-    <xacro:property name="triton_width"  value="0.5"/>
-    <xacro:property name="triton_height" value="0.5"/>
+    <xacro:property name="triton_length" value="0.25"/>
+    <xacro:property name="triton_width"  value="0.25"/>
+    <xacro:property name="triton_height" value="0.25"/>
     <xacro:macro name="triton_hydro_model" params="namespace">
       <!-- List of hydrodynamic models this robot's links -->
@@ -26,70 +26,7 @@
         <!-- Center of buoyancy -->
         <center_of_buoyancy>${triton_cob}</center_of_buoyancy>
-        <!--
-        Choose one of the hydrodynamic models below, all are based on
-        Fossen's equation of motion for underwater vehicles
-        Reference:
-        [1] Fossen, Thor I. Handbook of marine craft hydrodynamics and motion
-            control. John Wiley & Sons, 2011.
-        -->
-        <!-- 1) Fossen's equation of motion -->
-        <hydrodynamic_model>
-          <type>fossen</type>
-          <added_mass>
-            0 0 0 0 0 0
-            0 0 0 0 0 0
-            0 0 0 0 0 0
-            0 0 0 0 0 0
-            0 0 0 0 0 0
-            0 0 0 0 0 0
-          </added_mass>
-          <!--
-            The linear damping coefficients can be provided as a diagonal (6 elements)
-            or a full matrix (36 coefficients), like the added-mass coefficients above
-          -->
-          <linear_damping>
-            0 0 0 0 0 0
-          </linear_damping>
-          <!--
-            The linear damping coefficients proportional to the forward speed
-            can be provided as a diagonal (6 elements) or a full matrix (36 coefficients),
-            like the added-mass coefficients above.
-            This matrix is mostly useful for slender bodies (e.g. AUVs with torpedo shape)
-          -->
-          <linear_damping_forward_speed>
-            0 0 0 0 0 0
-          </linear_damping_forward_speed>
-          <!--
-            The quadratic damping coefficients can be provided as a diagonal (6 elements)
-            or a full matrix (36 coefficients), like the added-mass coefficients above
-          -->
-          <quadratic_damping>
-            0 0 0 0 0 0
-          </quadratic_damping>
-          <!--
-            In case you want to model a simple surface vessel, you can use the
-            implementation of linear (small angle) theory for boxed shaped vessels
-            by providing the following parameters. If you omit the area of the
-            water level plane area, it will be calculated from the bounding box
-            parameters. Uncomment the lines below in case you are simulating a
-            surface vessel.
-            For more details on these parameters and the computation of buoyancy
-            for vessels using this theory, check:
-              [1] Lecture Notes  TTK 4190 Guidance and Control of Vehicles (T. I. Fossen)
-                  http://www.fossen.biz/wiley/Ch4.pdf
-              [2] Fossen, Thor I. Handbook of marine craft hydrodynamics and motion
-                  control. John Wiley & Sons, 2011.
-          -->
-          <!--
-          <metacentric_width>0.0</metacentric_width>
-          <metacentric_length>0.0</metacentric_length>
-          <submerged_height>0.0</submerged_height>
-          -->
-        </hydrodynamic_model>
-        <!-- 2) This computes the added-mass and damping parameters for a sphere
-        in the fluid with the given radius -->
         <hydrodynamic_model>
           <type>sphere</type>
-          <radius>0</radius>
+          <radius>0.125</radius>
         </hydrodynamic_model>
       </link>

Commit message: Changed Joystick to a single launch for direct/setpoint mode Moved direct joystick controller matrix into controller matrix Created thrust odom to try to stabalize the EKF Added linear dampening to stablize Triton Adjusted Triton camera to closer to final parameters

File: cusub_sim/triton_description/urdf/base.xacro (robot description, xacro)
@@ -47,5 +47,5 @@
         </inertial>
         <visual>
-          <origin xyz="0 0 0" rpy="0 0 0"/>
+          <origin xyz="0 0 0" rpy="0 0 3.1415"/>
           <geometry>
             <mesh filename="${visual_mesh_file}" scale="1 1 1" />

File: cusub_sim/triton_description/urdf/gazebo.xacro (robot description, xacro)
@@ -27,7 +27,26 @@
         <center_of_buoyancy>${triton_cob}</center_of_buoyancy>
         <hydrodynamic_model>
+          <type>fossen</type>
+          <added_mass>
+           4.20515 0       0       0       0       0
+           0       4.20515 0       0       0       0
+           0       0       4.20515 0       0       0
+           0       0       0       0       0       0
+           0       0       0       0       0       0
+           0       0       0       0       0       0
+          </added_mass>
+          <linear_damping>
+            -1 -1 -1 -1 -1 -1
+          </linear_damping>
+          <quadratic_damping>
+            -12.6155 -12.6155 -12.6155 0 0 0
+          </quadratic_damping>
+        </hydrodynamic_model>
+        <!--
+        <hydrodynamic_model>
           <type>sphere</type>
           <radius>0.125</radius>
         </hydrodynamic_model>
+        -->
       </link>
     </xacro:macro>

File: cusub_sim/triton_description/urdf/sensors.xacro (robot description, xacro)
@@ -19,6 +19,6 @@
   <!-- Mount a camera  -->
   <xacro:ocam_camera_macro robot_namespace="${namespace}" camera_id="0" frame="ocam0_frame">
-    <axis xyz="0 0 0" />
-    <origin xyz="0.06 0 -0.05" rpy="0 -0.785398 0"/>
+    <axis xyz="0 0 1" />
+    <origin xyz="0.12 0 -0.04" rpy="0 0.6 0"/>
   </xacro:ocam_camera_macro>
 </robot>

File: cusub_sim/triton_description/urdf/snippets.xacro (robot description, xacro)
@@ -35,5 +35,6 @@
       <update_rate>30.0</update_rate>
       <camera name="rgb_camera">
-        <horizontal_fov>2.18166</horizontal_fov>
+        <!-- 100deg FOV -->
+        <horizontal_fov>1.74533</horizontal_fov>
         <image>
           <width>1280</width>
@@ -42,5 +43,5 @@
         </image>
         <clip>
-          <near>0.02</near>
+          <near>0.04</near>
           <far>300</far>
         </clip>

Commit message: Basic quad working

File: cusub_sim/triton_description/urdf/base.xacro (robot description, xacro)
@@ -15,5 +15,5 @@
   <xacro:property name="y_size"  value="0.25"/>
   <xacro:property name="z_size" value="0.25"/>
-  <xacro:property name="mass" value="3"/>
+  <xacro:property name="mass" value="4"/>
   <!-- Center of gravity -->
   <xacro:property name="cog" value="0 0 0"/>
