Commit message: Lazurus Functional

File: cusub_sim/triton_description/urdf/sensors.xacro (robot description, xacro)
@@ -15,5 +15,5 @@
   <!-- IMU  -->
   <xacro:default_imu namespace="${namespace}" parent_link="${namespace}/base_link">
-    <origin xyz="0 0 0" rpy="0 0 0"/>
+    <origin xyz="0 0 0" rpy="0 0 3.1415"/>
   </xacro:default_imu>
   <!-- Mount a camera  -->
