Commit message: Added torpedo despawn

File: cusub_sim/robosub_descriptions/models/Dropper/Dropper.xacro (robot description, xacro)
@@ -9,12 +9,12 @@
         rpy="0 0 0" />
       <mass
-        value="1.5" />
+        value="0.00412" />
         <inertia
-          ixx="0.01"
-          ixy="0.01"
-          ixz="0.01"
-          iyy="0.01"
-          iyz="0.01"
-          izz="0.01" />
+          ixx="0.00000004"
+          ixy="0.0"
+          ixz="0.0"
+          iyy="0.00000004"
+          iyz="0.0"
+          izz="0.00000004" />
       </inertial>
     <visual>
@@ -23,7 +23,7 @@
         rpy="0 0 0" />
       <geometry>
-        <sphere radius="0.01"/>
+        <sphere radius="0.005"/>
         <material name="black">
-          <color rgba="1 0.8 0 1"/>
+          <color rgba="0.2 0.2 0.2 1"/>
         </material>
       </geometry>
@@ -34,5 +34,5 @@
         rpy="0 0 0" />
       <geometry>
-        <sphere radius="0.01"/>
+        <sphere radius="0.005"/>
       </geometry>
     </collision>
@@ -47,9 +47,9 @@
         <flow_velocity_topic>hydrodynamics/current_velocity</flow_velocity_topic>
         <neutrally_buoyant>0</neutrally_buoyant>
-        <volume>0.001</volume>
+        <volume>0.000000524</volume>
         <box>
-          <width>0.1</width>
-          <length>0.1</length>
-          <height>0.1</height>
+          <width>0.01</width>
+          <length>0.01</length>
+          <height>0.01</height>
         </box>
         <!-- Center of buoyancy -->
@@ -57,5 +57,5 @@
         <hydrodynamic_model>
           <type>sphere</type>
-          <radius>0.25</radius>
+          <radius>0.005</radius>
         </hydrodynamic_model>
       </link>
