Commit message: Flipped z axis to Z up to NED nonsense problems with gazebo ros

File: cusub_sim/leviathan_description/urdf/snippets.xacro (robot description, xacro)
@@ -3,5 +3,5 @@
   <xacro:macro name="occam_camera_macro" params="robot_namespace camera_id frame *axis *origin">
   <!--camera_link-->
-  <link name="${robot_namespace}/camera_${camera_id}">
+  <link name="${robot_namespace}/${frame}">
     <collision>
       <origin xyz="0 0 0" rpy="0 0 0"/>
@@ -26,7 +26,7 @@
     <xacro:insert_block name="origin" />
     <parent link="${namespace}/base_link"/>
-    <child link="${robot_namespace}/camera_${camera_id}"/>
+    <child link="${robot_namespace}/${frame}"/>
   </joint>
-  <gazebo reference="${robot_namespace}/camera_${camera_id}">
+  <gazebo reference="${robot_namespace}/${frame}">
     <sensor type="camera" name="rgb_camera">
       <update_rate>30.0</update_rate>
@@ -76,5 +76,5 @@
   <xacro:macro name="downcam_camera_macro" params="robot_namespace camera_id frame *axis *origin">
   <!--camera_link-->
-  <link name="${robot_namespace}/camera_${camera_id}">
+  <link name="${robot_namespace}/${frame}">
     <collision>
       <origin xyz="0 0 0" rpy="0 0 0"/>
@@ -99,7 +99,7 @@
     <xacro:insert_block name="origin" />
     <parent link="${namespace}/base_link"/>
-    <child link="${robot_namespace}/camera_${camera_id}"/>
+    <child link="${robot_namespace}/${frame}"/>
   </joint>
-  <gazebo reference="${robot_namespace}/camera_${camera_id}">
+  <gazebo reference="${robot_namespace}/${frame}">
     <sensor type="camera" name="rgb_camera">
       <update_rate>30.0</update_rate>

Commit message: Fixed merge mistakes

File: cusub_sim/leviathan_description/urdf/snippets.xacro (robot description, xacro)
@@ -76,9 +76,5 @@
   <xacro:macro name="downcam_camera_macro" params="robot_namespace camera_id frame *axis *origin">
   <!--camera_link-->
-<<<<<<< HEAD
-  <link name="${robot_namespace}/camera_${camera_id}">
-=======
   <link name="${robot_namespace}/${frame}">
->>>>>>> 234fa89
     <collision>
       <origin xyz="0 0 0" rpy="0 0 0"/>

Commit message: Improved simulator for training data generation
Added torpedo model
Tweaked transdec surface so fog blends better
Added hydrodynamimcs to torpedos and droppers
Changed dice to be textured
Added visibility parameter for fake yolo
Tuned start gate pole points for bounding box in fake yolo
Added camera sensor noise
Updated TRANSDEC launch
Fixed dropper control in joy node

File: cusub_sim/leviathan_description/urdf/snippets.xacro (robot description, xacro)
@@ -49,4 +49,9 @@
           <far>300</far>
         </clip>
+        <noise>
+          <type>gaussian</type>
+          <mean>0.0</mean>
+          <stddev>0.008</stddev>
+        </noise>
         <distortion>
           <k1>-0.360085</k1>

File: cusub_sim/robosub_descriptions/models/Dice1/Dice1.xacro (robot description, xacro)
@@ -23,5 +23,5 @@
       <origin
         xyz="0 0 0"
-        rpy="1.5707963267949 0 0" />
+        rpy="0 0 0" />
       <geometry>
         <mesh
@@ -32,5 +32,5 @@
       <origin
         xyz="0 0 0"
-        rpy="1.5707963267949 0 0" />
+        rpy="0 0 0" />
       <geometry>
         <mesh

File: cusub_sim/robosub_descriptions/models/Dice5/Dice5.xacro (robot description, xacro)
@@ -23,5 +23,5 @@
       <origin
         xyz="0 0 0"
-        rpy="1.5707963267949 0 0" />
+        rpy="0 0 0" />
       <geometry>
         <mesh
@@ -32,5 +32,5 @@
       <origin
         xyz="0 0 0"
-        rpy="1.5707963267949 0 0" />
+        rpy="0 0 0" />
       <geometry>
         <mesh

File: cusub_sim/robosub_descriptions/models/Torpedo/Torpedo.xacro (robot description, xacro)
@@ -1,7 +1,7 @@
 <?xml version="1.0"?>
 <robot xmlns:xacro="http://www.ros.org/wiki/xacro"
-  name="Dropper_robot">
+  name="Torpedo_robot">
   <link
-    name="Dropper/base_link">
+    name="Torpedo/base_link">
     <inertial>
       <origin
@@ -9,30 +9,29 @@
         rpy="0 0 0" />
       <mass
-        value="1.5" />
+        value="0.0444" />
         <inertia
-          ixx="0.01"
-          ixy="0.01"
-          ixz="0.01"
-          iyy="0.01"
-          iyz="0.01"
-          izz="0.01" />
+          ixx="0.00003"
+          ixy="0.0"
+          ixz="0.0"
+          iyy="0.00003"
+          iyz="0.0"
+          izz="0.0" />
       </inertial>
     <visual>
       <origin
-        xyz="0 0 0"
+        xyz="0 0 -0.0629"
         rpy="0 0 0" />
       <geometry>
-        <sphere radius="0.01"/>
-        <material name="black">
-          <color rgba="1 0.8 0 1"/>
-        </material>
+        <mesh
+          filename="package://robosub_descriptions/models/Torpedo/Torpedo.stl" />
       </geometry>
     </visual>
     <collision>
       <origin
-        xyz="0 0 0"
+        xyz="0 0 -0.0629"
         rpy="0 0 0" />
       <geometry>
-        <sphere radius="0.01"/>
+        <mesh
+          filename="package://robosub_descriptions/models/Torpedo/Torpedo.stl" />
       </geometry>
     </collision>
@@ -43,19 +42,29 @@
     <flow_velocity_topic>hydrodynamics/current_velocity</flow_velocity_topic>
     <debug>0</debug>
-    <link name="Dropper/base_link">
+    <link name="Torpedo/base_link">
         <fluid_density>1028</fluid_density>
         <flow_velocity_topic>hydrodynamics/current_velocity</flow_velocity_topic>
         <neutrally_buoyant>0</neutrally_buoyant>
-        <volume>0.001</volume>
+        <volume>0.00004</volume>
         <box>
-          <width>0.1</width>
-          <length>0.1</length>
-          <height>0.1</height>
+          <width>0.025</width>
+          <length>0.117</length>
+          <height>0.025</height>
         </box>
         <!-- Center of buoyancy -->
         <center_of_buoyancy>0 0 0</center_of_buoyancy>
         <hydrodynamic_model>
-          <type>sphere</type>
-          <radius>0.25</radius>
+            <type>fossen</type>
+            <added_mass>
+              0    0    0    0     0    0
+              0    0    0    0     0    0
+              0    0    0    0     0    0
+              0    0    0    0     0    0
+              0    0    0    0     0    0
+              0    0    0    0     0    0
+            </added_mass>
+            <linear_damping>
+              -0.12 -0.12 -0.02 0 0 0
+            </linear_damping>
         </hydrodynamic_model>
       </link>

Commit message: Added optical frame for correct cv transforms Added ar tag models to divewell Added ar tag tracking and EKF

File: cusub_sim/leviathan_description/urdf/snippets.xacro (robot description, xacro)
@@ -2,4 +2,14 @@
 <robot xmlns:xacro="http://www.ros.org/wiki/xacro">
   <xacro:macro name="occam_camera_macro" params="robot_namespace camera_id frame *axis *origin">
+  <joint name="${robot_namespace}/camera_${camera_id}_optical_joint" type="fixed">
+    <!-- these values have to be these values otherwise the gazebo camera
+        image won't be aligned properly with the frame it is supposedly
+        originating from -->
+    <origin xyz="0 0 0" rpy="${-pi/2} 0 ${-pi/2}"/>
+    <parent link="${robot_namespace}/${frame}"/>
+    <child link="${robot_namespace}/${frame}_optical"/>
+  </joint>
+  <link name="${robot_namespace}/${frame}_optical">
+  </link>
   <!--camera_link-->
   <link name="${robot_namespace}/${frame}">
@@ -69,5 +79,5 @@
         <imageTopicName>image_raw</imageTopicName>
         <cameraInfoTopicName>camera_info</cameraInfoTopicName>
-        <frameName>${frame}</frameName>
+        <frameName>${frame}_optical</frameName>
         <distortionK1>-0.360085</distortionK1>
         <distortionK2>0.115116</distortionK2>

Commit message: Median averaging in mapper
rejects outliers and follows trends much better

File: cusub_sim/leviathan_description/urdf/snippets.xacro (robot description, xacro)
@@ -173,10 +173,10 @@
         </geometry>
       </visual>
-      <collision>
+      <!-- <collision>
         <origin xyz="0 0 0" rpy="0 1.5707963 0"/>
         <geometry>
           <cylinder radius="0.046" length="0.04"/>
         </geometry>
-      </collision>
+      </collision> -->
       <inertial>
         <mass value="0.001" />
