Commit message: Added gripper to leviathan

File: cusub_sim/leviathan_description/urdf/actuators.xacro (robot description, xacro)
@@ -49,3 +49,268 @@
     <origin xyz="-0.453136 -0.007874 -0.060706" rpy="0 0 -1.5707963" />
     </xacro:thruster_macro>
+  <link
+    name="${namespace}/gripper_link">
+    <inertial>
+      <origin
+        xyz="-3.05026979665671E-05 2.29258765859729E-10 0.129332205902841"
+        rpy="0 0 0" />
+      <mass
+        value="0.0685200444942305" />
+      <inertia
+        ixx="5.09046218363978E-05"
+        ixy="2.90940254882255E-15"
+        ixz="1.40373996687203E-07"
+        iyy="5.09050089301083E-05"
+        iyz="-1.05505321507431E-12"
+        izz="3.87093710476453E-10" />
+    </inertial>
+    <visual>
+      <origin
+        xyz="0 0 0"
+        rpy="0 0 0" />
+      <geometry>
+        <mesh
+          filename="package://leviathan_description/meshes/gripper_link.stl" />
+      </geometry>
+      <material
+        name="">
+        <color
+          rgba="0.1 0.1 0.1 1" />
+      </material>
+    </visual>
+    <collision>
+      <origin
+        xyz="0 0 0"
+        rpy="0 0 0" />
+      <geometry>
+        <mesh
+          filename="package://leviathan_description/meshes/gripper_link.stl" />
+      </geometry>
+    </collision>
+  </link>
+  <link
+    name="${namespace}/gripper/inner_link">
+    <inertial>
+      <origin
+        xyz="-2.49994954249532E-05 -0.00573643081918815 0.0251275882803392"
+        rpy="0 0 0" />
+      <mass
+        value="0.0120633523009251" />
+      <inertia
+        ixx="0"
+        ixy="0"
+        ixz="0"
+        iyy="0"
+        iyz="0"
+        izz="0" />
+    </inertial>
+    <visual>
+      <origin
+        xyz="0 0 0"
+        rpy="0 0 0" />
+      <geometry>
+        <mesh
+          filename="package://leviathan_description/meshes/inner_link.stl" />
+      </geometry>
+      <material
+        name="">
+        <color
+          rgba="0.1 0.1 0.1 1" />
+      </material>
+    </visual>
+    <collision>
+      <origin
+        xyz="0 0 0"
+        rpy="0 0 0" />
+      <geometry>
+        <mesh
+          filename="package://leviathan_description/meshes/inner_link.stl" />
+      </geometry>
+    </collision>
+  </link>
+  <joint
+    name="${namespace}/gripper/inner_joint"
+    type="revolute">
+    <origin
+      xyz="0 -0.2080920000001 0.02"
+      rpy="1.64478052298944 0 0" />
+    <parent
+      link="${namespace}/gripper_link" />
+    <child
+      link="${namespace}/gripper/inner_link" />
+    <axis
+      xyz="1 0 0" />
+    <limit
+      lower="-0.65"
+      upper="0.0"
+      effort="1"
+      velocity="1" />
+  </joint>
+  <!--
+  <link
+    name="${namespace}/gripper/pusher_link">
+    <inertial>
+      <origin
+        xyz="0.00011715199114278 1.32787251606671E-15 0.0375874379080091"
+        rpy="0 0 0" />
+      <mass
+        value="0.00592950115592324" />
+      <inertia
+        ixx="0"
+        ixy="0"
+        ixz="0"
+        iyy="0"
+        iyz="0"
+        izz="0" />
+    </inertial>
+    <visual>
+      <origin
+        xyz="0 0 0"
+        rpy="0 0 0" />
+      <geometry>
+        <mesh
+          filename="package://leviathan_description/meshes/pusher_link.stl" />
+      </geometry>
+      <material
+        name="">
+        <color
+          rgba="0.792156862745098 0.819607843137255 0.933333333333333 1" />
+      </material>
+    </visual>
+    <collision>
+      <origin
+        xyz="0 0 0"
+        rpy="0 0 0" />
+      <geometry>
+        <mesh
+          filename="package://leviathan_description/meshes/pusher_link.stl" />
+      </geometry>
+    </collision>
+  </link>
+  <joint
+    name="${namespace}/gripper/pusher_joint"
+    type="prismatic">
+    <origin
+      xyz="0 -0.144109728787135 0"
+      rpy="1.5707963267949 0 0" />
+    <parent
+      link="${namespace}/gripper_link" />
+    <child
+      link="${namespace}/gripper/pusher_link" />
+    <axis
+      xyz="0 0 1" />
+    <limit
+      lower="0.0"
+      upper="0.02"
+      effort="1"
+      velocity="1" />
+  </joint>-->
+  <link
+    name="${namespace}/gripper/outer_link">
+    <inertial>
+      <origin
+        xyz="-2.49973932494377E-05 0.00722026359518433 0.0253433707612258"
+        rpy="0 0 0" />
+      <mass
+        value="0.0145505838335253" />
+      <inertia
+        ixx="0"
+        ixy="0"
+        ixz="0"
+        iyy="0"
+        iyz="0"
+        izz="0" />
+    </inertial>
+    <visual>
+      <origin
+        xyz="0 0 0"
+        rpy="0 0 0" />
+      <geometry>
+        <mesh
+          filename="package://leviathan_description/meshes/outer_link.stl" />
+      </geometry>
+      <material
+        name="">
+        <color
+          rgba="0.1 0.1 0.1 1" />
+      </material>
+    </visual>
+    <collision>
+      <origin
+        xyz="0 0 0"
+        rpy="0 0 0" />
+      <geometry>
+        <mesh
+          filename="package://leviathan_description/meshes/outer_link.stl" />
+      </geometry>
+    </collision>
+  </link>
+  <joint
+    name="${namespace}/gripper/outer_joint"
+    type="revolute">
+    <origin
+      xyz="0 -0.2080920000001 -0.02"
+      rpy="1.49548129533638 0 0" />
+    <parent
+      link="${namespace}/gripper_link" />
+    <child
+      link="${namespace}/gripper/outer_link" />
+    <axis
+      xyz="1 0 0" />
+    <limit
+      lower="0.0"
+      upper="0.65"
+      effort="1"
+      velocity="1" />
+  </joint>
+  <transmission name="${namespace}/gripper/outer_transmission">
+    <type>transmission_interface/SimpleTransmission</type>
+      <joint name="${namespace}/gripper/outer_joint">
+        <hardwareInterface>hardware_interface/PositionJointInterface</hardwareInterface>
+      </joint>
+      <actuator name="${namespace}/gripper/outer_servo">
+        <hardwareInterface>hardware_interface/PositionJointInterface</hardwareInterface>
+        <mechanicalReduction>1</mechanicalReduction>
+      </actuator>
+  </transmission>
+  <transmission name="${namespace}/gripper/inner_transmission">
+    <type>transmission_interface/SimpleTransmission</type>
+      <joint name="${namespace}/gripper/inner_joint">
+        <hardwareInterface>hardware_interface/PositionJointInterface</hardwareInterface>
+      </joint>
+      <actuator name="${namespace}/gripper/inner_servo">
+        <hardwareInterface>hardware_interface/PositionJointInterface</hardwareInterface>
+        <mechanicalReduction>1</mechanicalReduction>
+      </actuator>
+  </transmission>
+  <gazebo reference="${namespace}/gripper_link">
+      <material>Gazebo/DarkGray</material>
+  </gazebo>
+  <gazebo reference="${namespace}/gripper/outer_link">
+      <material>Gazebo/DarkGray</material>
+  </gazebo>
+  <gazebo reference="${namespace}/gripper/inner_link">
+      <material>Gazebo/DarkGray</material>
+  </gazebo>
+  <gazebo>
+    <plugin name="gazebo_ros_control" filename="libgazebo_ros_control.so">
+      <robotNamespace>${namespace}</robotNamespace>
+    </plugin>
+  </gazebo>
+  <joint
+    name="${namespace}/gripper_joint"
+    type="fixed">
+    <origin
+      xyz="0.30 -0.14 -0.18"
+      rpy="0 1.57 1.57" />
+    <parent
+      link="${namespace}/base_link" />
+    <child
+      link="${namespace}/gripper_link" />
+    <axis
+      xyz="1 0 0" />
+    <limit
+      effort="0"
+      velocity="0" />
+  </joint>
 </robot>

File: cusub_sim/leviathan_description/urdf/sensors.xacro (robot description, xacro)
@@ -45,4 +45,8 @@
     <origin xyz="0 0 -0.1" rpy="0 1.57 0"/>
   </xacro:downcam_camera_macro>
+  <xacro:occam_camera_macro robot_namespace="${namespace}" camera_id="6" frame="gripper_cam_frame">
+    <axis xyz="0 0 1" />
+    <origin xyz="0.38 -0.14 -0.12" rpy="0 0.3 0"/>
+  </xacro:occam_camera_macro>
 <!--
   <xacro:regular_camera_plugin_macro

Commit message: Tweaked gripper to make yaw work again Started changing gripper to effort based added crucifix

File: cusub_sim/leviathan_description/urdf/actuators.xacro (robot description, xacro)
@@ -56,12 +56,12 @@
         rpy="0 0 0" />
       <mass
-        value="0.0685200444942305" />
+        value="0.001" />
       <inertia
-        ixx="5.09046218363978E-05"
-        ixy="2.90940254882255E-15"
-        ixz="1.40373996687203E-07"
-        iyy="5.09050089301083E-05"
-        iyz="-1.05505321507431E-12"
-        izz="3.87093710476453E-10" />
+        ixx="1.0E-5"
+        ixy="0.0"
+        ixz="0.0"
+        iyy="1.0E-5"
+        iyz="0.0"
+        izz="1.0E-5" />
     </inertial>
     <visual>
@@ -96,12 +96,12 @@
         rpy="0 0 0" />
       <mass
-        value="0.0120633523009251" />
+        value="0.001" />
       <inertia
-        ixx="0"
-        ixy="0"
-        ixz="0"
-        iyy="0"
-        iyz="0"
-        izz="0" />
+        ixx="1.0E-5"
+        ixy="0.0"
+        ixz="0.0"
+        iyy="1.0E-5"
+        iyz="0.0"
+        izz="1.0E-5" />
     </inertial>
     <visual>
@@ -147,63 +147,4 @@
       velocity="1" />
   </joint>
-  <!--
-  <link
-    name="${namespace}/gripper/pusher_link">
-    <inertial>
-      <origin
-        xyz="0.00011715199114278 1.32787251606671E-15 0.0375874379080091"
-        rpy="0 0 0" />
-      <mass
-        value="0.00592950115592324" />
-      <inertia
-        ixx="0"
-        ixy="0"
-        ixz="0"
-        iyy="0"
-        iyz="0"
-        izz="0" />
-    </inertial>
-    <visual>
-      <origin
-        xyz="0 0 0"
-        rpy="0 0 0" />
-      <geometry>
-        <mesh
-          filename="package://leviathan_description/meshes/pusher_link.stl" />
-      </geometry>
-      <material
-        name="">
-        <color
-          rgba="0.792156862745098 0.819607843137255 0.933333333333333 1" />
-      </material>
-    </visual>
-    <collision>
-      <origin
-        xyz="0 0 0"
-        rpy="0 0 0" />
-      <geometry>
-        <mesh
-          filename="package://leviathan_description/meshes/pusher_link.stl" />
-      </geometry>
-    </collision>
-  </link>
-  <joint
-    name="${namespace}/gripper/pusher_joint"
-    type="prismatic">
-    <origin
-      xyz="0 -0.144109728787135 0"
-      rpy="1.5707963267949 0 0" />
-    <parent
-      link="${namespace}/gripper_link" />
-    <child
-      link="${namespace}/gripper/pusher_link" />
-    <axis
-      xyz="0 0 1" />
-    <limit
-      lower="0.0"
-      upper="0.02"
-      effort="1"
-      velocity="1" />
-  </joint>-->
   <link
     name="${namespace}/gripper/outer_link">
@@ -213,12 +154,12 @@
         rpy="0 0 0" />
       <mass
-        value="0.0145505838335253" />
+        value="0.001" />
       <inertia
-        ixx="0"
-        ixy="0"
-        ixz="0"
-        iyy="0"
-        iyz="0"
-        izz="0" />
+        ixx="1.0E-5"
+        ixy="0.0"
+        ixz="0.0"
+        iyy="1.0E-5"
+        iyz="0.0"
+        izz="1.0E-5" />
     </inertial>
     <visual>
@@ -267,8 +208,8 @@
     <type>transmission_interface/SimpleTransmission</type>
       <joint name="${namespace}/gripper/outer_joint">
-        <hardwareInterface>hardware_interface/PositionJointInterface</hardwareInterface>
+        <hardwareInterface>hardware_interface/EffortJointInterface</hardwareInterface>
       </joint>
       <actuator name="${namespace}/gripper/outer_servo">
-        <hardwareInterface>hardware_interface/PositionJointInterface</hardwareInterface>
+        <hardwareInterface>hardware_interface/EffortJointInterface</hardwareInterface>
         <mechanicalReduction>1</mechanicalReduction>
       </actuator>
@@ -277,8 +218,8 @@
     <type>transmission_interface/SimpleTransmission</type>
       <joint name="${namespace}/gripper/inner_joint">
-        <hardwareInterface>hardware_interface/PositionJointInterface</hardwareInterface>
+        <hardwareInterface>hardware_interface/EffortJointInterface</hardwareInterface>
       </joint>
       <actuator name="${namespace}/gripper/inner_servo">
-        <hardwareInterface>hardware_interface/PositionJointInterface</hardwareInterface>
+        <hardwareInterface>hardware_interface/EffortJointInterface</hardwareInterface>
         <mechanicalReduction>1</mechanicalReduction>
       </actuator>

File: cusub_sim/leviathan_description/urdf/snippets.xacro (robot description, xacro)
@@ -90,4 +90,14 @@
   </xacro:macro>
   <xacro:macro name="downcam_camera_macro" params="robot_namespace camera_id frame *axis *origin">
+  <joint name="${robot_namespace}/camera_${camera_id}_optical_joint" type="fixed">
+    <!-- these values have to be these values otherwise the gazebo camera
+        image won't be aligned properly with the frame it is supposedly
+        originating from -->
+    <origin xyz="0 0 0" rpy="${-pi/2} 0 ${-pi/2}"/>
+    <parent link="${robot_namespace}/${frame}"/>
+    <child link="${robot_namespace}/${frame}_optical"/>
+  </joint>
+  <link name="${robot_namespace}/${frame}_optical">
+  </link>
   <!--camera_link-->
   <link name="${robot_namespace}/${frame}">
@@ -145,5 +155,5 @@
         <imageTopicName>image_raw</imageTopicName>
         <cameraInfoTopicName>camera_info</cameraInfoTopicName>
-        <frameName>${frame}</frameName>
+        <frameName>${frame}_optical</frameName>
         <distortionK1>0</distortionK1>
         <distortionK2>0</distortionK2>

Commit message: jiangshi autonomous
Former-commit-id: bd63c854c3e9611c9f99202b5d697cb385a54b85

File: cusub_sim/leviathan_description/urdf/actuators.xacro (robot description, xacro)
@@ -49,5 +49,5 @@
     <origin xyz="-0.453136 -0.007874 -0.060706" rpy="0 0 -1.5707963" />
     </xacro:thruster_macro>
-  <link
+  <!-- <link
     name="${namespace}/gripper_link">
     <inertial>
@@ -255,4 +255,4 @@
       effort="0"
       velocity="0" />
-  </joint>
+  </joint> -->
 </robot>

Commit message: add arm back to the sub

File: cusub_sim/leviathan_description/urdf/actuators.xacro (robot description, xacro)
@@ -49,5 +49,5 @@
     <origin xyz="-0.453136 -0.007874 -0.060706" rpy="0 0 -1.5707963" />
     </xacro:thruster_macro>
-  <!-- <link
+  <link
     name="${namespace}/gripper_link">
     <inertial>
@@ -244,5 +244,5 @@
     type="fixed">
     <origin
-      xyz="0.30 -0.14 -0.18"
+      xyz="0.30 -0.14 0"
       rpy="0 1.57 1.57" />
     <parent
@@ -255,4 +255,4 @@
       effort="0"
       velocity="0" />
-  </joint> -->
+  </joint>
 </robot>
