Commit message: Fake YOLO (#70)
* Inital Fake YOLO, have bounding boxes being generated with debug image for SG, and dice

Added distortion coefficents correctly to leviathan gazebo cameras
Moved start gate model top to be at origin
Added pose sensors to start gate and dice 5

* Changed levithan camera macros so we seperate the downcam
Inflated occam FoV to compensate for gazebo crop
Added publishing of darknet detections to FakeYOLO

* Cleand up YOLOFaker

Added camera info publishers to driver launch
Cleaned up yolo faker to be very parametric
Created YAML configuration for yolo faker for dice and start gate, added yaml for gazebo occam camera parameters
Added launch for yolo with yaml config passed to it
Added camera info publisher to give correct gazebo camera info to the yolo faker

* Inital Fake YOLO, have bounding boxes being generated with debug image for SG, and dice

Added distortion coefficents correctly to leviathan gazebo cameras
Moved start gate model top to be at origin
Added pose sensors to start gate and dice 5

* Changed levithan camera macros so we seperate the downcam
Inflated occam FoV to compensate for gazebo crop
Added publishing of darknet detections to FakeYOLO

* Cleand up YOLOFaker

Added camera info publishers to driver launch
Cleaned up yolo faker to be very parametric
Created YAML configuration for yolo faker for dice and start gate, added yaml for gazebo occam camera parameters
Added launch for yolo with yaml config passed to it
Added camera info publisher to give correct gazebo camera info to the yolo faker

* rebased new directory structure

* Documented YOLOFaker
Moved Leviathan Gazebo Drivers to scripts foulder

* Fixed yolo faker bugs from commenting pep8 compliance
Fixed bugs with sim launch from resturcturing

* Fakeyolo handles all obstacles

Fixed downcam resolution in levithan
Moved gt camera transforms to fake yolo launch file for now
Added downcam camera info publisher
Added pathmarker and roulette to fake yolo
Added show points debug option
Added downcam to fakeyolo

File: cusub_sim/leviathan_description/urdf/sensors.xacro (robot description, xacro)
@@ -21,28 +21,28 @@
     <origin xyz="0 0 0" rpy="0 0 0"/>
   </xacro:default_imu>
-  <xacro:camera_macro robot_namespace="${namespace}" camera_id="0" frame="occam0_frame">
+  <xacro:occam_camera_macro robot_namespace="${namespace}" camera_id="0" frame="occam0_frame">
     <axis xyz="0 0 0" />
     <origin xyz="0.055 0 0.22" rpy="0 0 0"/>
-  </xacro:camera_macro>
-  <xacro:camera_macro robot_namespace="${namespace}" camera_id="1" frame="occam1_frame">
+  </xacro:occam_camera_macro>
+  <xacro:occam_camera_macro robot_namespace="${namespace}" camera_id="1" frame="occam1_frame">
     <axis xyz="0 0 1" />
     <origin xyz="0.0169 -0.0523 0.22" rpy="0 0 -1.2566370"/>
-  </xacro:camera_macro>
-  <xacro:camera_macro robot_namespace="${namespace}" camera_id="2" frame="occam2_frame">
+  </xacro:occam_camera_macro>
+  <xacro:occam_camera_macro robot_namespace="${namespace}" camera_id="2" frame="occam2_frame">
     <axis xyz="0 0 1" />
     <origin xyz="-0.0444 -0.0323 0.22" rpy="0 0 -2.5132741"/>
-  </xacro:camera_macro>
-  <xacro:camera_macro robot_namespace="${namespace}" camera_id="3" frame="occam3_frame">
+  </xacro:occam_camera_macro>
+  <xacro:occam_camera_macro robot_namespace="${namespace}" camera_id="3" frame="occam3_frame">
     <axis xyz="0 0 1" />
     <origin xyz="-0.0444 0.0323 0.22" rpy="0 0 -3.7699111"/>
-  </xacro:camera_macro>
-  <xacro:camera_macro robot_namespace="${namespace}" camera_id="4" frame="occam4_frame">
+  </xacro:occam_camera_macro>
+  <xacro:occam_camera_macro robot_namespace="${namespace}" camera_id="4" frame="occam4_frame">
     <axis xyz="0 0 1" />
     <origin xyz="0.0169 0.0523 0.22" rpy="0 0 -5.0265482"/>
-  </xacro:camera_macro>
-  <xacro:camera_macro robot_namespace="${namespace}" camera_id="5" frame="downcam_frame">
+  </xacro:occam_camera_macro>
+  <xacro:downcam_camera_macro robot_namespace="${namespace}" camera_id="5" frame="downcam_frame">
     <axis xyz="0 0 1" />
     <origin xyz="0 0 -0.1" rpy="0 1.57 0"/>
-  </xacro:camera_macro>
+  </xacro:downcam_camera_macro>
 <!--
   <xacro:regular_camera_plugin_macro

File: cusub_sim/leviathan_description/urdf/snippets.xacro (robot description, xacro)
@@ -1,5 +1,5 @@
 <?xml version="1.0"?>
 <robot xmlns:xacro="http://www.ros.org/wiki/xacro">
-  <xacro:macro name="camera_macro" params="robot_namespace camera_id frame *axis *origin">
+  <xacro:macro name="occam_camera_macro" params="robot_namespace camera_id frame *axis *origin">
   <!--camera_link-->
   <link name="${robot_namespace}/camera_${camera_id}">
@@ -32,6 +32,12 @@
       <update_rate>30.0</update_rate>
       <camera name="rgb_camera">
-        <horizontal_fov>1.0397</horizontal_fov>
-        <vertical_fov>0.6443</vertical_fov>
+        <!--
+          The correct FOV is 1.0397, but because of gazebo distortion crop we
+           need to inflate it by 20% so it ends up the correct size
+          This will unfortunatly make it report a faulty camera matrix
+          TODO see if camera intrinsics propertys are working maybe we
+           can override
+        -->
+        <horizontal_fov>1.24764</horizontal_fov>
         <image>
           <width>752</width>
@@ -43,4 +49,12 @@
           <far>300</far>
         </clip>
+        <distortion>
+          <k1>-0.360085</k1>
+          <k2>0.115116</k2>
+          <k3>0.0</k3>
+          <p1>0.007768</p1>
+          <p2>0.004616</p2>
+          <center>0.5 0.5</center>
+        </distortion>
       </camera>
       <plugin name="camera_controller" filename="libgazebo_ros_camera.so">
@@ -51,10 +65,75 @@
         <cameraInfoTopicName>camera_info</cameraInfoTopicName>
         <frameName>${frame}</frameName>
-        <hackBaseline>0.0</hackBaseline>
         <distortionK1>-0.360085</distortionK1>
         <distortionK2>0.115116</distortionK2>
-        <distortionK3>0.007768</distortionK3>
-        <distortionT1>0.004616</distortionT1>
-        <distortionT2>0.000000</distortionT2>
+        <distortionK3>0.000000</distortionK3>
+        <distortionT1>0.007768</distortionT1>
+        <distortionT2>0.004616</distortionT2>
+      </plugin>
+    </sensor>
+  </gazebo>
+  </xacro:macro>
+  <xacro:macro name="downcam_camera_macro" params="robot_namespace camera_id frame *axis *origin">
+  <!--camera_link-->
+  <link name="${robot_namespace}/camera_${camera_id}">
+    <collision>
+      <origin xyz="0 0 0" rpy="0 0 0"/>
+      <geometry>
+        <!--mesh filename="package://simple_arm/meshes/camera.dae"/-->
+        <sphere radius="0.01"/>
+      </geometry>
+    </collision>
+    <visual>
+      <origin xyz="0 0 0" rpy="0 0 0"/>
+      <geometry>
+        <!--mesh filename="package://simple_arm/meshes/camera.dae"/-->
+        <sphere radius="0.01"/>
+      </geometry>
+      <material name="red">
+        <color rgba="1.0 0 0 1.0"/>
+      </material>
+    </visual>
+  </link>
+  <joint name="${robot_namespace}/camera_${camera_id}_joint" type="fixed">
+    <xacro:insert_block name="axis" />
+    <xacro:insert_block name="origin" />
+    <parent link="${namespace}/base_link"/>
+    <child link="${robot_namespace}/camera_${camera_id}"/>
+  </joint>
+  <gazebo reference="${robot_namespace}/camera_${camera_id}">
+    <sensor type="camera" name="rgb_camera">
+      <update_rate>30.0</update_rate>
+      <camera name="rgb_camera">
+        <horizontal_fov>2.18166</horizontal_fov>
+        <image>
+          <width>1280</width>
+          <height>960</height>
+          <format>R8G8B8</format>
+        </image>
+        <clip>
+          <near>0.02</near>
+          <far>300</far>
+        </clip>
+        <distortion>
+          <k1>0</k1>
+          <k2>0</k2>
+          <k3>0</k3>
+          <p1>0</p1>
+          <p2>0</p2>
+          <center>0.5 0.5</center>
+        </distortion>
+      </camera>
+      <plugin name="camera_controller" filename="libgazebo_ros_camera.so">
+        <alwaysOn>true</alwaysOn>
+        <updateRate>0.0</updateRate>
+        <cameraName>camera_${camera_id}</cameraName>
+        <imageTopicName>image_raw</imageTopicName>
+        <cameraInfoTopicName>camera_info</cameraInfoTopicName>
+        <frameName>${frame}</frameName>
+        <distortionK1>0</distortionK1>
+        <distortionK2>0</distortionK2>
+        <distortionK3>0</distortionK3>
+        <distortionT1>0</distortionT1>
+        <distortionT2>0</distortionT2>
       </plugin>
     </sensor>

File: cusub_sim/robosub_descriptions/models/PathMarker/PathMarker.xacro (robot description, xacro)
@@ -1,6 +1,10 @@
-<robot
+<?xml version="1.0"?>
+<robot xmlns:xacro="http://www.ros.org/wiki/xacro"
   name="PathMarker_robot">
+<!-- Loading file with sensor macros -->
+<xacro:include filename="$(find uuv_sensor_ros_plugins)/urdf/sensor_snippets.xacro"/>
+<xacro:macro name="pathmarker" params="namespace">
   <link
-    name="PathMarker_link">
+    name="${namespace}/base_link">
     <inertial>
       <origin
@@ -36,6 +40,9 @@
     </collision>
   </link>
-  <gazebo reference="PathMarker_link">
+  <xacro:default_pose_3d namespace="${namespace}" parent_link="${namespace}/base_link" />
+  <gazebo reference="${namespace}/base_link">
       <turnGravityOff>false</turnGravityOff>
   </gazebo>
+</xacro:macro>
+<xacro:pathmarker namespace="$(arg namespace)"/>
 </robot>

File: cusub_sim/robosub_descriptions/models/Roulette/Roulette.xacro (robot description, xacro)
@@ -1,6 +1,10 @@
-<robot
+<?xml version="1.0"?>
+<robot xmlns:xacro="http://www.ros.org/wiki/xacro"
   name="Roulette_robot">
+<!-- Loading file with sensor macros -->
+<xacro:include filename="$(find uuv_sensor_ros_plugins)/urdf/sensor_snippets.xacro"/>
+<xacro:macro name="roulette" params="namespace">
   <link
-    name="Roulette_link">
+    name="${namespace}/base_link">
     <inertial>
       <origin
@@ -36,6 +40,9 @@
     </collision>
   </link>
-  <gazebo reference="Roulette_link">
+  <xacro:default_pose_3d namespace="${namespace}" parent_link="${namespace}/base_link" />
+  <gazebo reference="${namespace}/base_link">
       <turnGravityOff>false</turnGravityOff>
   </gazebo>
+</xacro:macro>
+<xacro:roulette namespace="$(arg namespace)"/>
 </robot>

File: cusub_sim/robosub_descriptions/models/StartGate/StartGate.xacro (robot description, xacro)
@@ -1,6 +1,10 @@
-<robot
+<?xml version="1.0"?>
+<robot xmlns:xacro="http://www.ros.org/wiki/xacro"
   name="StartGate_robot">
+<!-- Loading file with sensor macros -->
+<xacro:include filename="$(find uuv_sensor_ros_plugins)/urdf/sensor_snippets.xacro"/>
+<xacro:macro name="startgate_base" params="namespace">
   <link
-    name="StartGate_link">
+    name="${namespace}/base_link">
     <inertial>
       <origin
@@ -34,6 +38,12 @@
     </collision>
   </link>
-  <gazebo reference="StartGate_link">
+  <xacro:default_pose_3d namespace="${namespace}" parent_link="${namespace}/base_link" />
+  <gazebo reference="${namespace}/base_link">
       <turnGravityOff>true</turnGravityOff>
   </gazebo>
+  <gazebo>
+      <static>true</static>
+  </gazebo>
+</xacro:macro>
+<xacro:startgate_base namespace="$(arg namespace)"/>
 </robot>

Commit message: Real sub fixes predive

File: cusub_sim/leviathan_description/urdf/sensors.xacro (robot description, xacro)
@@ -11,5 +11,5 @@
   <!-- DVL  -->
   <xacro:default_dvl namespace="${namespace}" parent_link="${namespace}/base_link">
-    <origin xyz="0 0 0" rpy="0 0 0"/>
+    <origin xyz="0 0 0" rpy="1.57 0 0"/>
   </xacro:default_dvl>
   <!-- Pressure  -->

Commit message: sub common launch now has robot state publisher and robot description 	TODO need joint state publisher to deal with non fixed links for dvl/imu 	TODO IMU needs to be changed to Z UP 	Also added occam launch and depth frame pub Fixed occam onecame launch to correct frame Fixed DVL rotation for sub in URDF

File: cusub_sim/leviathan_description/urdf/sensors.xacro (robot description, xacro)
@@ -11,5 +11,5 @@
   <!-- DVL  -->
   <xacro:default_dvl namespace="${namespace}" parent_link="${namespace}/base_link">
-    <origin xyz="0 0 0" rpy="1.57 0 0"/>
+    <origin xyz="0 0 0" rpy="0 0 1.57"/>
   </xacro:default_dvl>
   <!-- Pressure  -->

Commit message: Disabled pitch and roll in joy Changed occam to optical frame Added pitch roll pid config Updated localzer to new detection method

File: cusub_sim/leviathan_description/urdf/sensors.xacro (robot description, xacro)
@@ -11,5 +11,5 @@
   <!-- DVL  -->
   <xacro:default_dvl namespace="${namespace}" parent_link="${namespace}/base_link">
-    <origin xyz="0 0 0" rpy="0 0 0"/>
+    <origin xyz="0 0 0" rpy="0 0 1.57"/>
   </xacro:default_dvl>
   <!-- Pressure  -->

Commit message: Setup bundle AR detection Added camera launchs to sub launch Reenabled pitch control in joystick inverted cleaned up spartan driver a bit Tuned pitch Rotated IMU

File: cusub_sim/leviathan_description/urdf/sensors.xacro (robot description, xacro)
@@ -19,5 +19,5 @@
   <!-- IMU  -->
   <xacro:default_imu namespace="${namespace}" parent_link="${namespace}/base_link">
-    <origin xyz="0 0 0" rpy="0 0 0"/>
+    <origin xyz="0 0 0" rpy="0 0 -1.57"/>
   </xacro:default_imu>
   <xacro:occam_camera_macro robot_namespace="${namespace}" camera_id="0" frame="occam0_frame">

Commit message: Unreal FUN!

File: cusub_sim/leviathan_description/urdf/sensors.xacro (robot description, xacro)
@@ -9,60 +9,3 @@
   <!-- Mount a Pose 3D sensor. -->
   <xacro:default_pose_3d namespace="${namespace}" parent_link="${namespace}/base_link" />
-  <!-- DVL  -->
-  <xacro:default_dvl namespace="${namespace}" parent_link="${namespace}/base_link">
-    <origin xyz="0 0 0" rpy="0 0 1.57"/>
-  </xacro:default_dvl>
-  <!-- Pressure  -->
-  <xacro:default_pressure namespace="${namespace}" parent_link="${namespace}/base_link">
-    <origin xyz="0 0 0" rpy="0 0 0"/>
-  </xacro:default_pressure>
-  <!-- IMU  -->
-  <xacro:default_imu namespace="${namespace}" parent_link="${namespace}/base_link">
-    <origin xyz="0 0 0" rpy="0 0 -1.57"/>
-  </xacro:default_imu>
-  <xacro:occam_camera_macro robot_namespace="${namespace}" camera_id="0" frame="occam0_frame">
-    <axis xyz="0 0 0" />
-    <origin xyz="0.055 0 0.22" rpy="0 0 0"/>
-  </xacro:occam_camera_macro>
-  <xacro:occam_camera_macro robot_namespace="${namespace}" camera_id="1" frame="occam1_frame">
-    <axis xyz="0 0 1" />
-    <origin xyz="0.0169 -0.0523 0.22" rpy="0 0 -1.2566370"/>
-  </xacro:occam_camera_macro>
-  <xacro:occam_camera_macro robot_namespace="${namespace}" camera_id="2" frame="occam2_frame">
-    <axis xyz="0 0 1" />
-    <origin xyz="-0.0444 -0.0323 0.22" rpy="0 0 -2.5132741"/>
-  </xacro:occam_camera_macro>
-  <xacro:occam_camera_macro robot_namespace="${namespace}" camera_id="3" frame="occam3_frame">
-    <axis xyz="0 0 1" />
-    <origin xyz="-0.0444 0.0323 0.22" rpy="0 0 -3.7699111"/>
-  </xacro:occam_camera_macro>
-  <xacro:occam_camera_macro robot_namespace="${namespace}" camera_id="4" frame="occam4_frame">
-    <axis xyz="0 0 1" />
-    <origin xyz="0.0169 0.0523 0.22" rpy="0 0 -5.0265482"/>
-  </xacro:occam_camera_macro>
-  <xacro:downcam_camera_macro robot_namespace="${namespace}" camera_id="5" frame="downcam_frame">
-    <axis xyz="0 0 1" />
-    <origin xyz="0 0 -0.1" rpy="0 1.57 0"/>
-  </xacro:downcam_camera_macro>
-  <xacro:occam_camera_macro robot_namespace="${namespace}" camera_id="6" frame="gripper_cam_frame">
-    <axis xyz="0 0 1" />
-    <origin xyz="0.38 -0.14 -0.12" rpy="0 0.3 0"/>
-  </xacro:occam_camera_macro>
-<!--
-  <xacro:regular_camera_plugin_macro
-       namespace="${namespace}"
-       suffix=""
-       parent_link="${namespace}/base_link"
-       topic="camera"
-       mass="0.0015"
-       update_rate="15"
-       hfov="1.8125"
-       width="768"
-       height="492"
-       stddev="0.02"
-       scale="0.5">
-       <inertia ixx="0.0" ixy="0.0" ixz="0.0" iyy="0.00" iyz="0.0" izz="0.0" />
-       <origin xyz="0.0 0.2 0.0" rpy="0 0 1.5707963"/>
-   </xacro:regular_camera_plugin_macro>
--->
 </robot>

File: cusub_sim/robosub_descriptions/models/Torpedo/Torpedo.xacro (robot description, xacro)
@@ -2,6 +2,8 @@
 <robot xmlns:xacro="http://www.ros.org/wiki/xacro"
   name="Torpedo_robot">
+  <xacro:include filename="$(find uuv_sensor_ros_plugins)/urdf/sensor_snippets.xacro"/>
+  <xacro:macro name="torpedo_base" params="namespace">
   <link
-    name="Torpedo/base_link">
+    name="${namespace}/base_link">
     <inertial>
       <origin
@@ -9,5 +11,5 @@
         rpy="0 0 0" />
       <mass
-        value="0.0444" />
+        value="44000.444" />
         <inertia
           ixx="0.00003"
@@ -37,4 +39,5 @@
     </collision>
   </link>
+  <xacro:default_pose_3d namespace="${namespace}" parent_link="${namespace}/base_link" />
   <gazebo>
     <plugin filename="libuuv_underwater_object_ros_plugin.so" name="uuv_plugin">
@@ -42,9 +45,9 @@
     <flow_velocity_topic>hydrodynamics/current_velocity</flow_velocity_topic>
     <debug>0</debug>
-    <link name="Torpedo/base_link">
+    <link name="${namespace}/base_link">
         <fluid_density>1028</fluid_density>
         <flow_velocity_topic>hydrodynamics/current_velocity</flow_velocity_topic>
         <neutrally_buoyant>0</neutrally_buoyant>
-        <volume>0.00004</volume>
+        <volume>42.0</volume>
         <box>
           <width>0.025</width>
@@ -71,3 +74,5 @@
     </plugin>
   </gazebo>
+  </xacro:macro>
+  <xacro:torpedo_base namespace="$(arg namespace)"/>
 </robot>

Commit message: added torpedo cam

File: cusub_sim/leviathan_description/urdf/sensors.xacro (robot description, xacro)
@@ -49,4 +49,8 @@
     <origin xyz="0.38 -0.14 -0.12" rpy="0 0.3 0"/>
   </xacro:occam_camera_macro>
+  <xacro:occam_camera_macro robot_namespace="${namespace}" camera_id="7" frame="torpedo_cam_frame">
+    <axis xyz="0 0 1" />
+    <origin xyz="0.35 0.0 0.1" rpy="0 0.0 0"/>
+  </xacro:occam_camera_macro>
 <!--
   <xacro:regular_camera_plugin_macro

Commit message: Steredo down and torpedoes test

File: cusub_sim/leviathan_description/urdf/sensors.xacro (robot description, xacro)
@@ -21,4 +21,89 @@
     <origin xyz="0 0 0" rpy="0 0 -1.57"/>
   </xacro:default_imu>
+  <!-- PING  -->
+  <xacro:macro name="multibeam_sonar_2d"
+    params="namespace suffix parent_link topic mass update_rate
+      samples fov range_min range_max range_stddev mesh
+      *inertia *origin *visual">
+    <!-- Sensor link -->
+    <link name="${namespace}/sonar${suffix}_link">
+      <inertial>
+        <xacro:insert_block name="inertia" />
+        <mass value="${mass}" />
+        <origin xyz="0 0 0" rpy="0 0 0" />
+      </inertial>
+      <xacro:insert_block name="visual" />
+      <xacro:no_collision/>
+    </link>
+  <joint name="${namespace}_sonar${suffix}_joint" type="revolute">
+    <xacro:insert_block name="origin" />
+    <parent link="${parent_link}" />
+    <child link="${namespace}/sonar${suffix}_link" />
+    <limit upper="0" lower="0" effort="0" velocity="0" />
+    <axis xyz="1 0 0"/>
+  </joint>
+  <gazebo reference="${namespace}/sonar${suffix}_link">
+    <sensor type="gpu_ray" name="sonar${suffix}">
+      <pose>0 0 0 0 0 0</pose>
+      <visualize>false</visualize>
+      <update_rate>${update_rate}</update_rate>
+      <ray>
+        <scan>
+          <horizontal>
+            <samples>${samples}</samples>
+            <resolution>1</resolution>
+            <min_angle>-${0.5*fov}</min_angle>
+            <max_angle>${0.5*fov}</max_angle>
+          </horizontal>
+          <vertical>
+            <samples>${samples}</samples>
+            <resolution>1</resolution>
+            <min_angle>-${0.5*fov}</min_angle>
+            <max_angle> ${0.5*fov}</max_angle>
+          </vertical>
+        </scan>
+        <range>
+          <min>${range_min}</min>
+          <max>${range_max}</max>
+          <resolution>0.01</resolution>
+        </range>
+        <noise>
+          <type>gaussian</type>
+          <mean>0.0</mean>
+          <stddev>${range_stddev}</stddev>
+        </noise>
+      </ray>
+      <plugin name="sonar${suffix}_controller" filename="libgazebo_ros_velodyne_gpu_laser.so">
+        <topicName>${topic}</topicName>
+        <frameName>sonar${suffix}_link</frameName>
+          <min_range>${range_min}</min_range>
+          <max_range>${range_max}</max_range>
+          <gaussianNoise>0.0</gaussianNoise>
+      </plugin>
+    </sensor>
+  </gazebo>
+  </xacro:macro>
+  <xacro:multibeam_sonar_2d
+    namespace="${namespace}"
+    suffix=""
+    parent_link="${namespace}/base_link"
+    topic="sonar"
+    mass="0.02"
+    update_rate="15"
+    samples="32"
+    fov="0.523599"
+    range_min="1.0"
+    range_max="30.0"
+    range_stddev="0.027"
+    mesh="">
+    <inertia ixx="0.00001" ixy="0.0" ixz="0.0" iyy="0.00001" iyz="0.0" izz="0.00001" />
+    <origin xyz="0 0 0" rpy="0 0 0.0"/>
+    <visual>
+      <geometry>
+        <mesh filename="file://$(find uuv_sensor_ros_plugins)/meshes/p900.dae" scale="1 1 1"/>
+      </geometry>
+    </visual>
+    </xacro:multibeam_sonar_2d>
+  <!--
   <xacro:occam_camera_macro robot_namespace="${namespace}" camera_id="0" frame="occam0_frame">
     <axis xyz="0 0 0" />
@@ -52,4 +137,13 @@
     <axis xyz="0 0 1" />
     <origin xyz="0.35 0.0 0.1" rpy="0 0.0 0"/>
+  </xacro:occam_camera_macro>-->
+  <!-- Stereo Down -->
+  <xacro:occam_camera_macro robot_namespace="${namespace}" camera_id="8" frame="stereo_down_left_cam_frame">
+    <axis xyz="0 0 1" />
+    <origin xyz="0.0  0.05 -0.1" rpy="0 1.57 0"/>
+  </xacro:occam_camera_macro>
+  <xacro:occam_camera_macro robot_namespace="${namespace}" camera_id="9" frame="stereo_down_right_cam_frame">
+    <axis xyz="0 0 1" />
+    <origin xyz="0.0 -0.05 -0.1" rpy="0 1.57 0"/>
   </xacro:occam_camera_macro>
 <!--
