Commit message: Finish transdec
Former-commit-id: 67c6073cdfe6e3177c333c38f4b629e87b209a51

File: cusub_sim/robosub_descriptions/models/Octagon/Octagon.xacro (robot description, xacro)
@@ -1,14 +1,14 @@
 <?xml version="1.0"?>
 <robot xmlns:xacro="http://www.ros.org/wiki/xacro"
-  name="dice1_robot">
+  name="octagon">
   <!-- Loading file with sensor macros -->
   <xacro:include filename="$(find uuv_sensor_ros_plugins)/urdf/sensor_snippets.xacro"/>
-  <xacro:macro name="dropper_garlic_base" params="namespace">
+  <xacro:macro name="octagon_base" params="namespace">
     <xacro:default_pose_3d namespace="${namespace}" parent_link="${namespace}/base_link" />
     <link name="${namespace}/base_link">
       <inertial>
         <origin
-          xyz="0.0 0.0 1.0"
-          rpy="0 1.57 0" />
+          xyz="0.0 0.0 0.0"
+          rpy="0 0 0" />
         <mass
           value="0.2" />
@@ -22,17 +22,11 @@
       </inertial>
       <visual>
-        <origin
-          xyz="0 0.5 0"
-          rpy="1.57 0 0" />
         <geometry>
-          <mesh filename="model://dropper_garlic/dropper_garlic.dae" />
+          <mesh filename="model://Octagon/Octagon.dae"/>
         </geometry>
       </visual>
       <collision>
-        <origin
-          xyz="0 0.5 0"
-          rpy="1.57 0 0" />
         <geometry>
-          <mesh filename="model://dropper_garlic/dropper_garlic.dae" />
+          <mesh filename="model://Octagon/Octagon.dae"/>
         </geometry>
       </collision>
@@ -42,4 +36,4 @@
     </gazebo>
   </xacro:macro>
-  <xacro:dropper_garlic_base namespace="$(arg namespace)"/>
+  <xacro:octagon_base namespace="$(arg namespace)"/>
 </robot>

File: cusub_sim/robosub_descriptions/models/coffin/coffin.xacro (robot description, xacro)
@@ -1,8 +1,8 @@
 <?xml version="1.0"?>
 <robot xmlns:xacro="http://www.ros.org/wiki/xacro"
-  name="dice1_robot">
+  name="coffin">
   <!-- Loading file with sensor macros -->
   <xacro:include filename="$(find uuv_sensor_ros_plugins)/urdf/sensor_snippets.xacro"/>
-  <xacro:macro name="dropper_garlic_base" params="namespace">
+  <xacro:macro name="coffin_base" params="namespace">
     <xacro:default_pose_3d namespace="${namespace}" parent_link="${namespace}/base_link" />
     <link name="${namespace}/base_link">
@@ -10,5 +10,5 @@
         <origin
           xyz="0.0 0.0 1.0"
-          rpy="0 1.57 0" />
+          rpy="0 0 0" />
         <mass
           value="0.2" />
@@ -22,17 +22,11 @@
       </inertial>
       <visual>
-        <origin
-          xyz="0 0.5 0"
-          rpy="1.57 0 0" />
         <geometry>
-          <mesh filename="model://dropper_garlic/dropper_garlic.dae" />
+          <mesh filename="model://coffin/coffin.dae" />
         </geometry>
       </visual>
       <collision>
-        <origin
-          xyz="0 0.5 0"
-          rpy="1.57 0 0" />
         <geometry>
-          <mesh filename="model://dropper_garlic/dropper_garlic.dae" />
+          <mesh filename="model://coffin/coffin.dae" />
         </geometry>
       </collision>
@@ -42,4 +36,4 @@
     </gazebo>
   </xacro:macro>
-  <xacro:dropper_garlic_base namespace="$(arg namespace)"/>
+  <xacro:coffin_base namespace="$(arg namespace)"/>
 </robot>
