Commit message: Added vampire to FAKE YOLO!
Former-commit-id: 50e73251e16b97d4441681b4a77e5cebc8b33913

File: cusub_sim/robosub_descriptions/models/vampire_stake/vampire_stake.xacro (robot description, xacro)
@@ -5,4 +5,5 @@
   <xacro:include filename="$(find uuv_sensor_ros_plugins)/urdf/sensor_snippets.xacro"/>
   <xacro:macro name="vampire_steak_base" params="namespace">
+    <xacro:default_pose_3d namespace="${namespace}" parent_link="${namespace}/base_link" />
     <link name="${namespace}/base_link">
       <inertial>
@@ -96,6 +97,6 @@
     </link>
     <joint name="${namespace}/magic_base_joint" type="fixed">
-        <child link="${namespace}/base_link"/>
-        <parent link="${namespace}/magic_base_link"/>
+        <child link="${namespace}/magic_base_link"/>
+        <parent link="${namespace}/base_link"/>
     </joint>
     <gazebo>
