Commit message: slay distance and buoy dynamics tuned in the sim

File: cusub_sim/robosub_descriptions/models/triangular_buoy/triangular_buoy.xacro (robot description, xacro)
@@ -31,5 +31,5 @@
       <mass
         value="1" />
-      <inertia ixx="0" ixy="0" ixz="0" iyy="0" iyz="0" izz="0" />
+      <inertia ixx="1" ixy="0" ixz="0" iyy="1" iyz="0" izz="1" />
     </inertial>
     <visual>

Commit message: triangular bouy fixes for xacro
Former-commit-id: 2121d3f75dd30e95f9bed6e002208dc982ba7881

File: cusub_sim/robosub_descriptions/models/triangular_buoy/triangular_buoy.xacro (robot description, xacro)
@@ -1,77 +1,85 @@
-<robot name="bouy_robot">
-  <link name="base_link">
-    <inertial>
-      <origin xyz="0 0 0" rpy="0 0 0" />
-      <mass value="20" />
-      <inertia ixx="0" ixy="0" ixz="0" iyy="0" iyz="0" izz="0" />
-    </inertial>
-    <visual>
+<?xml version="1.0"?>
+<robot xmlns:xacro="http://www.ros.org/wiki/xacro"
+  name="triangular_bouy_robot">
+  <!-- Loading file with sensor macros -->
+  <xacro:include filename="$(find uuv_sensor_ros_plugins)/urdf/sensor_snippets.xacro"/>
+  <xacro:macro name="triangular_buoy_base" params="namespace" >
+    <xacro:default_pose_3d namespace="${namespace}" parent_link="${namespace}/base_link" />
+    <link name="${namespace}/base_link">
+      <inertial>
+        <origin xyz="0 0 0" rpy="0 0 0" />
+        <mass value="20" />
+        <inertia ixx="0" ixy="0" ixz="0" iyy="0" iyz="0" izz="0" />
+      </inertial>
+      <visual>
+        <origin
+          xyz="0 0 0"
+          rpy="0 0 0" />
+        <geometry>
+          <box size="1.0 1.0 0.1"/>
+        </geometry>
+      </visual>
+      <collision>
+        <origin
+          xyz="0 0 0"
+          rpy="0 0 0" />
+        <geometry>
+          <box size="1.0 1.0 0.1"/>
+        </geometry>
+      </collision>
+    </link>
+    <link
+      name="${namespace}/buoy_link">
+      <inertial>
+        <origin
+          xyz="0 0.0 0"
+          rpy="0 0 0" />
+        <mass
+          value="1" />
+        <inertia ixx="1" ixy="0" ixz="0" iyy="1" iyz="0" izz="1" />
+      </inertial>
+      <visual>
+        <origin xyz="0 0 0" rpy="0 0.0 0" />
+        <geometry>
+          <mesh filename="package://robosub_descriptions/models/triangular_buoy/triangular_buoy.dae" />
+        </geometry>
+      </visual>
+      <collision>
+        <origin xyz="0 0 0" rpy="0 0.0 0" />
+        <geometry>
+          <mesh filename="package://robosub_descriptions/models/triangular_buoy/triangular_buoy.dae" />
+        </geometry>
+      </collision>
+    </link>
+    <joint
+      name="${namespace}/anchor_joint"
+      type="continuous">
       <origin
-        xyz="0 0 0"
+        xyz="0 0 2.5"
         rpy="0 0 0" />
-      <geometry>
-        <box size="1.0 1.0 0.1"/>
-      </geometry>
-    </visual>
-    <collision>
-      <origin
-        xyz="0 0 0"
-        rpy="0 0 0" />
-      <geometry>
-        <box size="1.0 1.0 0.1"/>
-      </geometry>
-    </collision>
-  </link>
-  <link
-    name="buoy_link">
-    <inertial>
-      <origin
-        xyz="0 0.0 0"
-        rpy="0 0 0" />
-      <mass
-        value="1" />
-      <inertia ixx="1" ixy="0" ixz="0" iyy="1" iyz="0" izz="1" />
-    </inertial>
-    <visual>
-      <origin xyz="0 0 0" rpy="0 0.0 0" />
-      <geometry>
-        <mesh filename="package://robosub_descriptions/models/triangular_buoy/triangular_buoy.dae" />
-      </geometry>
-    </visual>
-    <collision>
-      <origin xyz="0 0 0" rpy="0 0.0 0" />
-      <geometry>
-        <mesh filename="package://robosub_descriptions/models/triangular_buoy/triangular_buoy.dae" />
-      </geometry>
-    </collision>
-  </link>
-  <joint
-    name="anchor_joint"
-    type="continuous">
-    <origin
-      xyz="0 0 2.5"
-      rpy="0 0 0" />
-    <parent
-      link="base_link" />
-    <child
-      link="buoy_link" />
-    <axis xyz="0 0 1" />
-    <dynamics damping="0.0" friction="0.0"/>
-    <limit effort="1000.0" velocity="10.0" />
-  </joint>
-  <transmission name="anchor_transmission">
-    <type>transmission_interface/SimpleTransmission</type>
-      <joint name="anchor_joint">
-        <hardwareInterface>hardware_interface/VelocityJointInterface</hardwareInterface>
-      </joint>
-      <actuator name="anchor_servo">
-        <hardwareInterface>hardware_interface/VelocityJointInterface</hardwareInterface>
-        <mechanicalReduction>1</mechanicalReduction>
-      </actuator>
-  </transmission>
-  <gazebo>
-    <plugin name="gazebo_ros_control" filename="libgazebo_ros_control.so">
-      <robotNamespace>/triangular_buoy_1</robotNamespace>
-    </plugin>
-  </gazebo>
+      <parent
+        link="${namespace}/base_link" />
+      <child
+        link="${namespace}/buoy_link" />
+      <axis xyz="0 0 1" />
+      <dynamics damping="0.0" friction="0.0"/>
+      <limit effort="1000.0" velocity="10.0" />
+    </joint>
+    <transmission name="anchor_transmission">
+      <type>transmission_interface/SimpleTransmission</type>
+        <joint name="${namespace}/anchor_joint">
+          <hardwareInterface>hardware_interface/VelocityJointInterface</hardwareInterface>
+        </joint>
+        <actuator name="${namespace}/anchor_servo">
+          <hardwareInterface>hardware_interface/VelocityJointInterface</hardwareInterface>
+          <mechanicalReduction>1</mechanicalReduction>
+        </actuator>
+    </transmission>
+    <gazebo>
+      <plugin name="gazebo_ros_control" filename="libgazebo_ros_control.so">
+        <robotNamespace>/triangular_buoy_1</robotNamespace>
+      </plugin>
+    </gazebo>
+  </xacro:macro>
+  <xacro:triangular_buoy_base namespace="$(arg namespace)"/>
 </robot>

Commit message: Triangle Buoy works with fake YOLO
Former-commit-id: 1fa9e3e8b22c4166a75f825a9bd9ff8823001123

File: cusub_sim/robosub_descriptions/models/triangular_buoy/triangular_buoy.xacro (robot description, xacro)
@@ -5,5 +5,5 @@
   <xacro:include filename="$(find uuv_sensor_ros_plugins)/urdf/sensor_snippets.xacro"/>
   <xacro:macro name="triangular_buoy_base" params="namespace" >
-    <xacro:default_pose_3d namespace="${namespace}" parent_link="${namespace}/base_link" />
+    <xacro:default_pose_3d namespace="${namespace}" parent_link="${namespace}/buoy_link" />
     <link name="${namespace}/base_link">
       <inertial>
@@ -40,5 +40,5 @@
       </inertial>
       <visual>
-        <origin xyz="0 0 0" rpy="0 0.0 0" />
+        <origin xyz="0 0 0" rpy="0 0 0" />
         <geometry>
           <mesh filename="package://robosub_descriptions/models/triangular_buoy/triangular_buoy.dae" />
@@ -46,5 +46,5 @@
       </visual>
       <collision>
-        <origin xyz="0 0 0" rpy="0 0.0 0" />
+        <origin xyz="0 0 0" rpy="0 0 0" />
         <geometry>
           <mesh filename="package://robosub_descriptions/models/triangular_buoy/triangular_buoy.dae" />

Commit message: possibly dangerous but i need to merge with lazarus

File: cusub_sim/robosub_descriptions/models/triangular_buoy/triangular_buoy.xacro (robot description, xacro)
@@ -58,28 +58,68 @@
         xyz="0 0 2.5"
         rpy="0 0 0" />
-      <parent
-        link="${namespace}/base_link" />
-      <child
-        link="${namespace}/buoy_link" />
-      <axis xyz="0 0 1" />
-      <dynamics damping="0.0" friction="0.0"/>
-      <limit effort="1000.0" velocity="10.0" />
-    </joint>
-    <transmission name="anchor_transmission">
-      <type>transmission_interface/SimpleTransmission</type>
-        <joint name="${namespace}/anchor_joint">
-          <hardwareInterface>hardware_interface/VelocityJointInterface</hardwareInterface>
-        </joint>
-        <actuator name="${namespace}/anchor_servo">
-          <hardwareInterface>hardware_interface/VelocityJointInterface</hardwareInterface>
-          <mechanicalReduction>1</mechanicalReduction>
-        </actuator>
-    </transmission>
-    <gazebo>
-      <plugin name="gazebo_ros_control" filename="libgazebo_ros_control.so">
-        <robotNamespace>/triangular_buoy_1</robotNamespace>
-      </plugin>
-    </gazebo>
-  </xacro:macro>
-  <xacro:triangular_buoy_base namespace="$(arg namespace)"/>
+      <geometry>
+        <box size="1.0 1.0 0.1"/>
+      </geometry>
+    </visual>
+    <collision>
+      <origin
+        xyz="0 0 0"
+        rpy="0 0 0" />
+      <geometry>
+        <box size="1.0 1.0 0.1"/>
+      </geometry>
+    </collision>
+  </link>
+  <link
+    name="buoy_link">
+    <inertial>
+      <origin
+        xyz="0 0.0 0"
+        rpy="0 0 0" />
+      <mass
+        value="1" />
+      <inertia ixx="1" ixy="0" ixz="0" iyy="1" iyz="0" izz="1" />
+    </inertial>
+    <visual>
+      <origin xyz="0 0 0" rpy="0 0.0 0" />
+      <geometry>
+        <mesh filename="package://robosub_descriptions/models/triangular_buoy/triangular_buoy.dae" />
+      </geometry>
+    </visual>
+    <collision>
+      <origin xyz="0 0 0" rpy="0 0.0 0" />
+      <geometry>
+        <mesh filename="package://robosub_descriptions/models/triangular_buoy/triangular_buoy.dae" />
+      </geometry>
+    </collision>
+  </link>
+  <joint
+    name="anchor_joint"
+    type="continuous">
+    <origin
+      xyz="0 0 2.5"
+      rpy="0 0 0" />
+    <parent
+      link="base_link" />
+    <child
+      link="buoy_link" />
+    <axis xyz="0 0 1" />
+    <dynamics damping="0.0" friction="0.0"/>
+    <limit effort="1000.0" velocity="10.0" />
+  </joint>
+  <transmission name="anchor_transmission">
+    <type>transmission_interface/SimpleTransmission</type>
+      <joint name="anchor_joint">
+        <hardwareInterface>hardware_interface/VelocityJointInterface</hardwareInterface>
+      </joint>
+      <actuator name="anchor_servo">
+        <hardwareInterface>hardware_interface/VelocityJointInterface</hardwareInterface>
+        <mechanicalReduction>1</mechanicalReduction>
+      </actuator>
+  </transmission>
+  <gazebo>
+    <plugin name="gazebo_ros_control" filename="libgazebo_ros_control.so">
+      <robotNamespace>/triangular_buoy_1</robotNamespace>
+    </plugin>
+  </gazebo>
 </robot>
